File: hardware/trollbook.kicad_pcb (KiCad board)
At the start: 2 copper layers, 100 x 100 mm, 46 parts, among them P1 VGA, P2 LCD, P3 SPI, P4 CONN_12, P5 CONN_2, P6 CONN_2, P7 CONN_2, U1 XC95288-208, U10 74LS574, U11 74LS574, U12 HY57V561620, U13 HY57V561620, U15 74HC4002, U16 ADA4851-4, U19 74HC139, U2 MC68030, U20 74HC10, U3 MC68882, U4 IDT71V416, U5 TLC7524, U6 74LS574, U7 39F040, U8 TLC7524, U9 74LS574, Y1 50 MHz, Y2 12.288 MHz

Commit message: aaaaawww yeeeaaaahhh
Parts:
- added P10: CONN_1, PINTST, F.Cu at (98.8, 163.3)
- added P8: CONN_4, PIN_ARRAY_4x1, F.Cu at (184.3, 142.8)
- added P9: CONN_2, PIN_ARRAY_2X1, F.Cu at (91.6, 191.1)
- moved P4 87.4 mm to (155.6, 144.7), turned to 180 degrees
- moved P5 35.9 mm to (91.5, 214.1), turned to 270 degrees
- moved R8 31.5 mm to (103.6, 153.5), turned to 180 degrees
- moved R9 28.4 mm to (103.6, 155.5), turned to 180 degrees
- moved R5 26.0 mm to (101.2, 158.1), turned to 270 degrees
- moved R4 21.0 mm to (99.5, 158.0), turned to 90 degrees
- moved R6 18.6 mm to (96.3, 169.3), turned to 180 degrees
- moved P6 16.8 mm to (119.1, 147.3)
- moved R7 16.3 mm to (95.4, 160.8), turned to 90 degrees
- moved P7 8.21 mm to (142.8, 149.7)
- moved P3 8.18 mm to (158.1, 148.4)
- moved R1 1.14 mm to (96.3, 180.5)
Connections:
- P2 pad 44: (no net) -> N-00000106
- P2 pad 46: (no net) -> /VCOM
- P2 pad 6: (no net) -> /VCOM
- P4 pad 11: (no net) -> /VCOM
- P4 pad 5: +10V -> (no net)
Routing:
- net 3V3: track 16.4 -> 653.5 mm, vias 0 -> 42
- net +5V: track 7.88 -> 560.7 mm, vias 1 -> 34
- net GND: track 0.00 -> 361.0 mm, vias 0 -> 75
- net N-0000049: track 0.00 -> 110.4 mm, vias 0 -> 4
- net /RESET: track 0.00 -> 108.2 mm, vias 0 -> 4
- net /VCOM: track 0.00 -> 92.2 mm, vias 0 -> 3
- net +15V: track 0.00 -> 65.8 mm, vias 0 -> 3
- net -10V: track 0.00 -> 60.7 mm, vias 0 -> 3
- net N-0000061: track 0.00 -> 53.0 mm, vias 0 -> 2
- net N-0000062: track 0.00 -> 51.6 mm, vias 0 -> 2
- net N-0000063: track 0.00 -> 49.9 mm, vias 0 -> 3
- net /AS: track 6.87 -> 55.2 mm, vias 1 -> 4
- net /DSACK0: track 6.71 -> 55.0 mm, vias 1 -> 4
- net /DSACK1: track 6.92 -> 54.8 mm, vias 1 -> 4
- net /DS: track 8.42 -> 54.6 mm, vias 1 -> 4
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- added copper zone on B.Cu, net GND

Commit message: capacitors, capacitors everywhere
Parts:
- added C1: 1n, SM0805, B.Cu at (135.1, 211.6)
- added C10: 1n, SM0805, B.Cu at (141.9, 167.2)
- added C11: 100n, SM0805, B.Cu at (133.2, 211.6)
- added C12: 1n, SM0805, B.Cu at (164.6, 189.3)
- added C13: 100n, SM0805, F.Cu at (101.5, 205.8)
- added C14: 100n, SM0805, F.Cu at (122.4, 158.8)
- added C15: 100n, SM0805, F.Cu at (103.8, 149.6)
- added C16: 100n, SM0805, F.Cu at (188.1, 206.0)
- added C17: 100n, SM0805, B.Cu at (179.4, 202.6)
- added C18: 100n, SM0805, F.Cu at (157.4, 170.8)
- added C19: 100n, SM0805, B.Cu at (158.6, 205.4)
- added C2: 1n, SM0805, F.Cu at (158.6, 191.8)
- added C20: 100n, SM0805, B.Cu at (170.1, 172.0)
- added C21: 100n, SM0805, F.Cu at (127.6, 188.2)
- added C22: 100n, SM0805, B.Cu at (187.5, 184.9)
- added C23: 100n, SM0805, F.Cu at (186.7, 170.8)
- added C24: 100n, SM0805, B.Cu at (108.2, 181.7)
- added C25: 100n, SM0805, B.Cu at (120.2, 175.1)
- added C26: 100n, SM0805, B.Cu at (119.5, 200.2)
- added C27: 100n, SM0805, B.Cu at (120.0, 164.8)
- added C28: 100n, SM0805, B.Cu at (186.9, 209.6)
- added C29: 100n, SM0805, B.Cu at (180.9, 224.3)
- added C3: 1n, SM0805, B.Cu at (158.6, 209.2)
- added C30: 100n, SM0805, B.Cu at (158.3, 219.3)
- added C31: 100n, SM0805, F.Cu at (111.6, 218.9)
- added C32: 100n, SM0805, F.Cu at (112.9, 228.1)
- added C33: 100n, SM0805, F.Cu at (118.2, 150.6)
- added C34: 10u, SM1206, F.Cu at (136.3, 144.7)
- added C35: 10u, SM1206, F.Cu at (174.4, 146.7)
- added C36: 10u, SM1206, F.Cu at (167.6, 153.0)
- added C37: 10u, SM1206, F.Cu at (170.9, 150.4)
- added C38: 10u, SM1206, F.Cu at (138.9, 149.2)
- added C39: 10u, SM1206, F.Cu at (155.4, 147.3)
- added C4: 1n, SM0805, B.Cu at (124.3, 172.1)
- added C40: 10u, SM1206, F.Cu at (94.1, 191.3)
- added C41: 100n, SM0805, F.Cu at (149.5, 146.9)
- added C42: 100n, SM0805, F.Cu at (146.4, 149.2)
- added C43: 100n, SM0805, F.Cu at (96.3, 191.1)
- added C5: 100n, SM0805, B.Cu at (158.6, 207.3)
- added C6: 100n, SM0805, F.Cu at (141.0, 161.0)
- added C7: 100n, SM0805, B.Cu at (126.2, 170.5)
- added C8: 100n, SM0805, B.Cu at (124.9, 202.2)
- added C9: 100n, SM0805, B.Cu at (170.2, 170.2)
- moved R5 0.76 mm to (102.0, 158.0)
- moved R4 0.64 mm to (100.1, 158.0)
Routing:
- net GND: track 361.0 -> 418.6 mm, vias 75 -> 85
- net +5V: track 560.7 -> 609.3 mm
- net 3V3: track 653.5 -> 688.5 mm, vias 42 -> 43
- net +10V: track 8.69 -> 11.0 mm
- net N-0000024: track 8.37 -> 9.69 mm
- net N-000003: track 28.0 -> 29.3 mm
- net +15V: track 65.8 -> 67.0 mm
- net -10V: track 60.7 -> 61.6 mm
- net N-0000023: track 40.7 -> 41.4 mm
- net /RAMCAS: track 43.8 -> 43.3 mm
