File: hardware/trollbook.sch (KiCad schematic (older format))
At the start: 4 parts, among them U1 XC95288-208, U2 MC68030, U3 MC68882, U4 IDT71V416

Commit message: routed address and data lines between cpu, fpu, rom, cpld
Parts:
- added J1: DB15, symbol DB15
- added J2: VGAF, symbol VGAF
- added R1, R10, R11, R12, R13, R14, R15, R16, R2, R3, R4, R5, R6, R7, R8, R9: R, ~, symbol R
- added R17, R18, R19: 75, ~, symbol R
- added RP1, RP2, RP3, RP4: R_PACK4, ~, symbol R_PACK4
- added U5: 74LS244, ~, symbol 74LS244
- added U6: 74LS574, ~, symbol 74LS574
- added U7: 39F040, ~, symbol 39F040
- added U8: MCP660, symbol MCP660
- U4: footprint (none) -> ~
Connections:
- net labels added: +5V, 3V3, A0, A1, A10, A11, A12, A13, A14, A15, A16, A17, A18, A19, A2, A20, A21, A22, A23, A24, A25, A26, A27, A28, A29, A3, A30, A31, A4, A5, A6, A7, A8, A9, D0, D1, D10, D11, D12, D13, D14, D15, D16, D17, D18, D19, D2, D20, D21, D22, D23, D24, D25, D26, D27, D28, D29, D3, D30, D31, D4, D5, D6, D7, D8, D9, GND, LLA1, LLA10, LLA11, LLA12, LLA13, LLA14, LLA15, LLA16, LLA17, LLA18, LLA2, LLA3, LLA4, LLA5, LLA6, LLA7, LLA8, LLA9, LLBHE, LLBLE, LLCS, LLD0, LLD1, LLD10, LLD11, LLD12, LLD13, LLD14, LLD15, LLD2, LLD3, LLD4, LLD5, LLD6, LLD7, LLD8, LLD9, LLOE, LLWEN
- wire segments 0 -> 446
- no-connect marks 0 -> 4
Other:
- moved on the sheet: U1, U2, U3

Commit message: dram
Parts:
- removed J1: DB15, symbol DB15
- removed R10, R11, R12, R13, R14, R15, R16, R4, R5, R6, R7, R8, R9: R, ~, symbol R
- added RP5, RP6, RP7, RP8: 10k, ~, symbol R_PACK4
- added U10, U11, U9: 74LS574, ~, symbol 74LS574
- added U12, U13: HY57V561620, symbol HY57V561620
- added U?: OSC, symbol OSC
- R1, R2, R3: value R -> 10k
- RP1, RP2, RP3, RP4: value R_PACK4 -> 20k
Connections:
- net labels added: AS, AVEC, BERR, CBACK, CBREQ, CLK50, CPUCLK, DBEN, DS, DSACK0, DSACK1, FC0, FC1, FC2, FPUCS, IPEND, IPL0, IPL1, IPL2, RAMA0, RAMA1, RAMA10, RAMA11, RAMA12, RAMA2, RAMA3, RAMA4, RAMA5, RAMA6, RAMA7, RAMA8, RAMA9, RAMB0, RAMB1, RAMCAS, RAMCKE, RAMCLK, RAMCS0, RAMCS1, RAMD0, RAMD1, RAMD10, RAMD11, RAMD12, RAMD13, RAMD14, RAMD15, RAMD2, RAMD3, RAMD4, RAMD5, RAMD6, RAMD7, RAMD8, RAMD9, RAMLDQM, RAMRAS, RAMUDQM, RAMWE, RESET, ROMCE, ROMOE, RW, SIZ0, SIZ1, STERM, VGAB0, VGAB1, VGAB2, VGAB3, VGAB4, VGAG0, VGAG1, VGAG2, VGAG3, VGAG4, VGAG5, VGAR0, VGAR1, VGAR2, VGAR3, VGAR4
- wire segments 446 -> 630
- no-connect marks 4 -> 8
Other:
- note added: "B"
- note added: "G"
- note added: "R"
- moved on the sheet: R17, R18, R19, RP1, RP2, RP3, RP4, U6, U7

Commit message: routed sram, dram
Parts:
- removed J2: VGAF, symbol VGAF
- removed U5: 74LS244, ~, symbol 74LS244
- removed U8: MCP660, symbol MCP660
- removed U?: OSC, symbol OSC
- added K1: CONN_3, symbol CONN_3
- added P1: VGA, symbol CONN_6
- added P2: LCD, symbol CONN_50
- added P3: SPI, symbol CONN_8
- added U15: 74HC4002, symbol 74HC4002
- added U16: ADA4851-4, ~, symbol ADA4851-4
- added U17, U18: DAC0800, symbol DAC0800
- added U19: 74HC139, ~, symbol 74LS139
- added U20: 74HC10, ~, symbol 74LS10
- added Y1: 50 MHz, ~, symbol OSC
- added Y2: 12.288 MHz, ~, symbol OSC
Connections:
- net labels added: ATOOHIGH, CLK12, CPUMODE, EXTINT, SNDLATCH, SPICLK, SPIMISO, SPIMOSI, SPISS1, SPISS2, SPISS3, SPISS4, SSBIN0, SSBIN1, VGAHSYNC, VGALATCH, VGAOE, VGAVSYNC
- net labels removed: RAMCKE, RAMCLK
- wire segments 630 -> 732
Other:
- note added: "spi slave select"
- moved on the sheet: U11, U6, U9

Commit message: moved sram closer to cpu
Changed lines of the file:
@@
 Sheet 1 1
 Title ""
-Date "11 dec 2014"
+Date "12 dec 2014"
 Rev ""
 Comp ""
@@
 Text Label 4300 17700 0    60   ~ 0
 LLD5
+Text Label 4300 17500 0    60   ~ 0
+LLD6
 Text Label 4300 17600 0    60   ~ 0
-LLD6
-Text Label 4300 17500 0    60   ~ 0
 LLD7
 Text Label 4300 15700 0    60   ~ 0

Commit message: lcd connector, vga dac
Parts:
- removed K1: CONN_3, symbol CONN_3
- added P4: CONN_12, symbol CONN_12
- added P5, P6, P7: CONN_2, symbol CONN_2
- added R4, R5, R6: 560k, ~, symbol R
- added R7, R8, R9: 150k, ~, symbol R
Connections:
- net labels added: +10V, +15V, -10V
- wire segments 732 -> 829
- no-connect marks 8 -> 14

Commit message: ostkaka
Parts:
- removed U17, U18: DAC0800, symbol DAC0800
- added P8: CONN_4, symbol CONN_4
- added U5, U8: TLC7524, symbol TLC7524
Connections:
- wire segments 829 -> 843
- no-connect marks 14 -> 16

Commit message: aaaaawww yeeeaaaahhh
Parts:
- added P10: CONN_1, symbol CONN_1
- added P9: CONN_2, symbol CONN_2
Connections:
- net labels added: VCOM
- wire segments 843 -> 846
- no-connect marks 16 -> 17
Other:
- note added: "Retarded datasheet does\nnot specify polarity"
Changed lines of the file:
@@
 Sheet 1 1
 Title ""
-Date "9 jan 2015"
+Date "15 jan 2015"
 Rev ""
 Comp ""
@@
 $EndComp
 $Comp
-L CONN_12 P4
-U 1 1 548B9D74
-P 29850 10700
-F 0 "P4" V 29800 10700 60  0000 C CNN
-F 1 "CONN_12" V 29900 10700 60  0000 C CNN
-F 2 "" H 29850 10700 60  0000 C CNN
-F 3 "" H 29850 10700 60  0000 C CNN
-	1    29850 10700
-	0    -1   -1   0
-$EndComp
-$Comp
 L +10V #PWR061
 U 1 1 548B9D81
-P 29700 11150
-F 0 "#PWR061" H 29700 11400 30  0001 C CNN
-F 1 "+10V" H 29700 11350 30  0000 C CNN
-F 2 "" H 29700 11150 60  0000 C CNN
-F 3 "" H 29700 11150 60  0000 C CNN
-	1    29700 11150
+P 28300 11100
+F 0 "#PWR061" H 28300 11350 30  0001 C CNN
+F 1 "+10V" H 28300 11300 30  0000 C CNN
+F 2 "" H 28300 11100 60  0000 C CNN
+F 3 "" H 28300 11100 60  0000 C CNN
+	1    28300 11100
 	-1   0    0    1
 $EndComp
@@
 $EndComp
 $Comp
-L -10V #PWR91
+L -10V #PWR92
 U 1 1 548B9D8D
 P 30100 11200
-F 0 "#PWR91" H 30100 11330 20  0001 C CNN
+F 0 "#PWR92" H 30100 11330 20  0001 C CNN
 F 1 "-10V" H 30100 11300 30  0000 C CNN
 F 2 "" H 30100 11200 60  0000 C CNN
@@
 	1    0    0    -1
 $EndComp
-NoConn ~ 30300 11050
 $Comp
 L CONN_2 P7
@@
 	4750 8650 4000 8650
 Wire Wire Line
-	4750 8750 4000 8750
-Wire Wire Line
-	4750 8850 4000 8850
+	3050 8750 4750 8750
 Wire Wire Line
 	4750 8950 4000 8950
@@
 	29300 11100 29300 11050
 Wire Wire Line
-	29700 11150 29700 11050
-Wire Wire Line
 	29900 11150 29900 11050
 Wire Wire Line
@@
 	29900 5350 29900 4500
 Connection ~ 29500 5350
+$Comp
+L CONN_12 P4
+U 1 1 548B9D74
+P 29850 10700
+F 0 "P4" V 29800 10700 60  0000 C CNN
+F 1 "CONN_12" V 29900 10700 60  0000 C CNN
+F 2 "" H 29850 10700 60  0000 C CNN
+F 3 "" H 29850 10700 60  0000 C CNN
+	1    29850 10700
+	0    -1   -1   0
+$EndComp
+Wire Wire Line
+	30300 11050 30300 11350
+Wire Wire Line
+	30300 11350 30800 11350
+Text Label 30350 11350 0    60   ~ 0
+VCOM
+Text Label 4200 4950 0    60   ~ 0
+VCOM
+Text Label 4200 8950 0    60   ~ 0
+VCOM
+Text Notes 2250 9000 0    60   ~ 0
+Retarded datasheet does\nnot specify polarity
+$Comp
+L CONN_2 P9
+U 1 1 54B71211
+P 28200 10700
+F 0 "P9" V 28150 10700 40  0000 C CNN
+F 1 "CONN_2" V 28250 10700 40  0000 C CNN
+F 2 "" H 28200 10700 60  0000 C CNN
+F 3 "" H 28200 10700 60  0000 C CNN
+	1    28200 10700
+	0    -1   -1   0
+$EndComp
+$Comp
+L GND #PWR093
+U 1 1 54B7122A
+P 28100 11100
+F 0 "#PWR093" H 28100 11100 30  0001 C CNN
+F 1 "GND" H 28100 11030 30  0001 C CNN
+F 2 "" H 28100 11100 60  0000 C CNN
+F 3 "" H 28100 11100 60  0000 C CNN
+	1    28100 11100
+	1    0    0    -1
+$EndComp
+Wire Wire Line
+	28100 11100 28100 11050
+Wire Wire Line
+	28300 11100 28300 11050
+NoConn ~ 29700 11050
+$Comp
+L CONN_1 P10
+U 1 1 54B71EA6
+P 2900 8750
+F 0 "P10" H 2980 8750 40  0000 L CNN
+F 1 "CONN_1" H 2900 8805 30  0001 C CNN
+F 2 "" H 2900 8750 60  0000 C CNN
+F 3 "" H 2900 8750 60  0000 C CNN
+	1    2900 8750
+	-1   0    0    1
+$EndComp
+Wire Wire Line
+	4750 8850 4000 8850
+NoConn ~ 4000 8850
 $EndSCHEMATC

Commit message: capacitors, capacitors everywhere
Parts:
- added C1, C10, C12, C2, C3, C4: 1n, ~, symbol C
- added C11, C13, C14, C15, C16, C17, C18, C19, C20, C21, C22, C23, C24, C25, C26, C27, C28, C29, C30, C31, C32, C33, C41, C42, C43, C5, C6, C7, C8, C9: 100n, ~, symbol C
- added C34, C35, C36, C37, C38, C39, C40: 10u, ~, symbol C
Connections:
- wire segments 846 -> 910
