File: hardware/trollbook.sch (KiCad schematic (older format))
At the start: 92 parts, among them P1 VGA, P10 CONN_1, P2 LCD, P3 SPI, P4 CONN_12, P5 CONN_2, P6 CONN_2, P7 CONN_2, P8 CONN_4, P9 CONN_2, U1 XC95288-208, U10 74LS574, U11 74LS574, U12 HY57V561620, U13 HY57V561620, U15 74HC4002, U16 ADA4851-4, U19 74HC139, U2 MC68030, U20 74HC10, U3 MC68882, U4 IDT71V416, U5 TLC7524, U6 74LS574, U7 39F040, U8 TLC7524, U9 74LS574, Y1 50 MHz, Y2 12.288 MHz

Commit message: fixed some erc/drc violations
Parts:
- removed P2: LCD, symbol CONN_50
- added P11: CONN_2, symbol CONN_2
- added P2: LCD_CONN, ~, symbol LCD_CONN
Connections:
- wire segments 910 -> 918
- no-connect marks 17 -> 24
Changed lines of the file:
@@
 RAMUDQM
 $Comp
-L CONN_50 P2
-U 1 1 548AAD44
-P 5050 6850
-F 0 "P2" V 5250 6850 60  0000 C CNN
-F 1 "LCD" V 5150 6850 60  0000 C CNN
-F 2 "" H 5450 7950 60  0000 C CNN
-F 3 "" H 5450 7950 60  0000 C CNN
-	1    5050 6850
-	1    0    0    -1
-$EndComp
-$Comp
 L GND #PWR040
 U 1 1 548AC792
@@
 $EndComp
 $Comp
-L -10V #PWR124
+L -10V #PWR125
 U 1 1 548B9D8D
 P 30100 11200
-F 0 "#PWR124" H 30100 11330 20  0001 C CNN
+F 0 "#PWR125" H 30100 11330 20  0001 C CNN
 F 1 "-10V" H 30100 11300 30  0000 C CNN
 F 2 "" H 30100 11200 60  0000 C CNN
@@
 	8600 19200 9150 19200
 Wire Wire Line
-	8600 18500 9150 18500
+	8600 18500 9800 18500
 Wire Wire Line
 	1450 20100 1450 20000
@@
 $EndComp
 $Comp
-L -10V #PWR129
+L -10V #PWR130
 U 1 1 54B85D80
 P 30400 11900
-F 0 "#PWR129" H 30400 12030 20  0001 C CNN
+F 0 "#PWR130" H 30400 12030 20  0001 C CNN
 F 1 "-10V" H 30400 12000 30  0000 C CNN
 F 2 "" H 30400 11900 60  0000 C CNN
@@
 Wire Wire Line
 	31500 12400 31300 12400
+NoConn ~ 10650 8050
+NoConn ~ 14100 7200
+NoConn ~ 14100 7400
+NoConn ~ 14100 7600
+NoConn ~ 14100 7800
+Wire Wire Line
+	12400 6950 12400 7750
+Connection ~ 12400 7400
+Wire Wire Line
+	12400 6950 12800 6950
+Connection ~ 12800 6950
+Connection ~ 12400 7250
+Connection ~ 11750 8100
+Connection ~ 11750 8000
+Wire Wire Line
+	11750 7900 11750 8450
+Wire Wire Line
+	11750 8450 11300 8450
+Wire Wire Line
+	11300 8450 11300 8550
+Connection ~ 11750 8200
+NoConn ~ 19600 10850
+NoConn ~ 15150 10950
+$Comp
+L CONN_2 P11
+U 1 1 54B8235F
+P 10150 18600
+F 0 "P11" V 10100 18600 40  0000 C CNN
+F 1 "CONN_2" V 10200 18600 40  0000 C CNN
+F 2 "" H 10150 18600 60  0000 C CNN
+F 3 "" H 10150 18600 60  0000 C CNN
+	1    10150 18600
+	1    0    0    -1
+$EndComp
+Wire Wire Line
+	9800 18700 9750 18700
+Wire Wire Line
+	9750 18700 9750 18850
+$Comp
+L GND #PWR0133
+U 1 1 54B82BE0
+P 9750 18850
+F 0 "#PWR0133" H 9750 18850 30  0001 C CNN
+F 1 "GND" H 9750 18780 30  0001 C CNN
+F 2 "" H 9750 18850 60  0000 C CNN
+F 3 "" H 9750 18850 60  0000 C CNN
+	1    9750 18850
+	1    0    0    -1
+$EndComp
+$Comp
+L LCD_CONN P2
+U 1 1 54B84A6E
+P 5050 6850
+F 0 "P2" V 5250 6850 60  0000 C CNN
+F 1 "LCD_CONN" V 5150 6850 60  0000 C CNN
+F 2 "~" H 5450 7950 60  0000 C CNN
+F 3 "~" H 5450 7950 60  0000 C CNN
+	1    5050 6850
+	1    0    0    -1
+$EndComp
+$Comp
+L GND #PWR?
+U 1 1 54B84EAE
+P 5150 9800
+F 0 "#PWR?" H 5150 9800 30  0001 C CNN
+F 1 "GND" H 5150 9730 30  0001 C CNN
+F 2 "" H 5150 9800 60  0000 C CNN
+F 3 "" H 5150 9800 60  0000 C CNN
+	1    5150 9800
+	1    0    0    -1
+$EndComp
+Wire Wire Line
+	5150 9800 5150 9750
 $EndSCHEMATC

Commit message: arne
Parts:
- added R10, R11, R12, R13: 10k, ~, symbol R
Connections:
- wire segments 918 -> 924
Other:
- moved on the sheet: P8
Changed lines of the file:
@@
 Sheet 1 1
 Title ""
-Date "15 jan 2015"
+Date "17 jan 2015"
 Rev ""
 Comp ""
@@
 $EndComp
 $Comp
-L -10V #PWR23
+L -10V #PWR61
 U 1 1 548B81B6
 P 4000 8550
-F 0 "#PWR23" H 4000 8680 20  0001 C CNN
+F 0 "#PWR61" H 4000 8680 20  0001 C CNN
 F 1 "-10V" H 4000 8650 30  0000 C CNN
 F 2 "" H 4000 8550 60  0000 C CNN
@@
 $EndComp
 $Comp
-L -10V #PWR125
+L -10V #PWR85
 U 1 1 548B9D8D
 P 30100 11200
-F 0 "#PWR125" H 30100 11330 20  0001 C CNN
+F 0 "#PWR85" H 30100 11330 20  0001 C CNN
 F 1 "-10V" H 30100 11300 30  0000 C CNN
 F 2 "" H 30100 11200 60  0000 C CNN
@@
 L CONN_4 P8
 U 1 1 54A5A241
-P 4100 18800
-F 0 "P8" V 4050 18800 50  0000 C CNN
-F 1 "CONN_4" V 4150 18800 50  0000 C CNN
-F 2 "" H 4100 18800 60  0000 C CNN
-F 3 "" H 4100 18800 60  0000 C CNN
-	1    4100 18800
+P 2750 18800
+F 0 "P8" V 2700 18800 50  0000 C CNN
+F 1 "CONN_4" V 2800 18800 50  0000 C CNN
+F 2 "" H 2750 18800 60  0000 C CNN
+F 3 "" H 2750 18800 60  0000 C CNN
+	1    2750 18800
 	-1   0    0    1
 $EndComp
@@
 	6900 3900 6900 3800
 Wire Wire Line
-	4600 18650 4450 18650
+	3100 18650 4600 18650
 Wire Wire Line
-	4600 18750 4450 18750
+	3100 18750 4600 18750
 Wire Wire Line
-	4600 18850 4450 18850
+	3100 18850 4600 18850
 Wire Wire Line
-	4600 18950 4450 18950
+	3100 18950 4600 18950
 Wire Wire Line
 	26600 3650 26600 3350
@@
 $EndComp
 $Comp
-L -10V #PWR130
+L -10V #PWR94
 U 1 1 54B85D80
 P 30400 11900
-F 0 "#PWR130" H 30400 12030 20  0001 C CNN
+F 0 "#PWR94" H 30400 12030 20  0001 C CNN
 F 1 "-10V" H 30400 12000 30  0000 C CNN
 F 2 "" H 30400 11900 60  0000 C CNN
@@
 $EndComp
 $Comp
-L GND #PWR?
+L GND #PWR0134
 U 1 1 54B84EAE
 P 5150 9800
-F 0 "#PWR?" H 5150 9800 30  0001 C CNN
+F 0 "#PWR0134" H 5150 9800 30  0001 C CNN
 F 1 "GND" H 5150 9730 30  0001 C CNN
 F 2 "" H 5150 9800 60  0000 C CNN
@@
 Wire Wire Line
 	5150 9800 5150 9750
+$Comp
+L R R10
+U 1 1 54BAB187
+P 3150 18350
+F 0 "R10" V 3230 18350 40  0000 C CNN
+F 1 "10k" V 3157 18351 40  0000 C CNN
+F 2 "~" V 3080 18350 30  0000 C CNN
+F 3 "~" H 3150 18350 30  0000 C CNN
+	1    3150 18350
+	1    0    0    -1
+$EndComp
+$Comp
+L R R11
+U 1 1 54BAB1AB
+P 3300 18350
+F 0 "R11" V 3380 18350 40  0000 C CNN
+F 1 "10k" V 3307 18351 40  0000 C CNN
+F 2 "~" V 3230 18350 30  0000 C CNN
+F 3 "~" H 3300 18350 30  0000 C CNN
+	1    3300 18350
+	1    0    0    -1
+$EndComp
+$Comp
+L R R12
+U 1 1 54BAB1B1
+P 3450 18350
+F 0 "R12" V 3530 18350 40  0000 C CNN
+F 1 "10k" V 3457 18351 40  0000 C CNN
+F 2 "~" V 3380 18350 30  0000 C CNN
+F 3 "~" H 3450 18350 30  0000 C CNN
+	1    3450 18350
+	1    0    0    -1
+$EndComp
+$Comp
+L R R13
+U 1 1 54BAB1B7
+P 3600 18350
+F 0 "R13" V 3680 18350 40  0000 C CNN
+F 1 "10k" V 3607 18351 40  0000 C CNN
+F 2 "~" V 3530 18350 30  0000 C CNN
+F 3 "~" H 3600 18350 30  0000 C CNN
+	1    3600 18350
+	1    0    0    -1
+$EndComp
+$Comp
+L 3V3 #PWR0135
+U 1 1 54BAB1BF
+P 3150 18000
+F 0 "#PWR0135" H 3150 18100 40  0001 C CNN
+F 1 "3V3" H 3150 18125 40  0000 C CNN
+F 2 "" H 3150 18000 60  0000 C CNN
+F 3 "" H 3150 18000 60  0000 C CNN
+	1    3150 18000
+	1    0    0    -1
+$EndComp
+Wire Wire Line
+	3150 18000 3150 18100
+Wire Wire Line
+	3150 18100 3600 18100
+Connection ~ 3300 18100
+Connection ~ 3450 18100
+Wire Wire Line
+	3150 18600 3150 18650
+Connection ~ 3150 18650
+Wire Wire Line
+	3300 18600 3300 18750
+Connection ~ 3300 18750
+Wire Wire Line
+	3450 18600 3450 18850
+Connection ~ 3450 18850
+Wire Wire Line
+	3600 18600 3600 18950
+Connection ~ 3600 18950
 $EndSCHEMATC

Commit message: fixed a couple of voltage issues
Parts:
- U10, U11, U6, U9: value 74LS574 -> 74LVC574
- U20: value 74HC10 -> 74LVC10
