File: hardware-rev2/trollbook-rev2.sch (KiCad schematic (older format))
At the start: 1 part

Commit message: cpu footprint
Parts:
- U1: renamed from U?; footprint MODULE -> mod:QFP-184
Changed lines of the file:
@@
 $EndDescr
 $Comp
-L MC68040FC33V U?
+L MC68040FC33V U1
 U 1 1 55DD5ACC
 P 15300 10500
-F 0 "U?" H 15300 10450 50  0000 C CNN
+F 0 "U1" H 15300 10450 50  0000 C CNN
 F 1 "MC68040FC33V" H 15300 10550 50  0000 C CNN
-F 2 "MODULE" H 15300 10100 50  0001 C CNN
+F 2 "mod:QFP-184" H 15300 10100 50  0001 C CNN
 F 3 "DOCUMENTATION" H 15300 10000 50  0001 C CNN
 	1    15300 10500

Commit message: added fpga
Parts:
- added U2: EPF10K50VRC240, mod:RQFP-240, symbol EPF10K50VRC240
Other:
- moved on the sheet: U1
Changed lines of the file:
@@
 LIBS:valves
 LIBS:MC68040FC33V
+LIBS:EPF10K50VRC240
 LIBS:trollbook-rev2-cache
 EELAYER 25 0
@@
 L MC68040FC33V U1
 U 1 1 55DD5ACC
-P 15300 10500
-F 0 "U1" H 15300 10450 50  0000 C CNN
-F 1 "MC68040FC33V" H 15300 10550 50  0000 C CNN
-F 2 "mod:QFP-184" H 15300 10100 50  0001 C CNN
-F 3 "DOCUMENTATION" H 15300 10000 50  0001 C CNN
-	1    15300 10500
+P 21550 11800
+F 0 "U1" H 21550 11750 50  0000 C CNN
+F 1 "MC68040FC33V" H 21550 11850 50  0000 C CNN
+F 2 "mod:QFP-184" H 21550 11400 50  0001 C CNN
+F 3 "DOCUMENTATION" H 21550 11300 50  0001 C CNN
+	1    21550 11800
 	1    0    0    -1
 $EndComp
+$Comp
+L EPF10K50VRC240 U2
+U 1 1 55DEFDF4
+P 10000 11600
+F 0 "U2" H 10000 11550 50  0000 C CNN
+F 1 "EPF10K50VRC240" H 10000 11650 50  0000 C CNN
+F 2 "mod:RQFP-240" H 10000 11100 50  0001 C CNN
+F 3 "DOCUMENTATION" H 10000 11000 50  0001 C CNN
+	1    10000 11600
+	1    0    0    -1
+$EndComp

Commit message: fixed clearance, added ram
Parts:
- added U3: 39F040, symbol 39F040
- added U4, U5: HY57V561620, mod:TSOP54, symbol HY57V561620
- added U6: IDT71V416, mod:TSOP44, symbol IDT71V416
- added U7, U8: TLC7524, Housings_SOIC:SOIC-16_3.9x9.9mm_Pitch1.27mm, symbol TLC7524
Connections:
- net labels added: +3V3, A0, A1, A10, A11, A12, A13, A14, A15, A16, A17, A18, A19, A2, A20, A21, A22, A23, A24, A25, A26, A27, A28, A29, A3, A30, A31, A4, A5, A6, A7, A8, A9, D0, D1, D10, D11, D12, D13, D14, D15, D16, D17, D18, D19, D2, D20, D21, D22, D23, D24, D25, D26, D27, D28, D29, D3, D30, D31, D4, D5, D6, D7, D8, D9, GND
- wire segments 0 -> 104

Commit message: arne
Parts:
- removed U6: IDT71V416, mod:TSOP44, symbol IDT71V416
- added CON? (x2): AVR-JTAG-10, AVR-JTAG-10, symbol AVR-JTAG-10
- added P?: CONN_01X02, symbol CONN_01X02
- added R? (x5): 10k, symbol R
Connections:
- net labels added: CLK33, LLA1, LLA10, LLA11, LLA12, LLA13, LLA14, LLA15, LLA16, LLA17, LLA18, LLA2, LLA3, LLA4, LLA5, LLA6, LLA7, LLA8, LLA9, LLD0, LLD1, LLD10, LLD11, LLD12, LLD13, LLD14, LLD15, LLD2, LLD3, LLD4, LLD5, LLD6, LLD7, LLD8, LLD9, ROMD0, ROMD1, ROMD2, ROMD3, ROMD4, ROMD5, ROMD6, ROMD7
- wire segments 104 -> 267
- no-connect marks 0 -> 3
Other:
- moved on the sheet: U3, U5

Commit message: started connecting processor to glue
Parts:
- added P1: CONN_01X01, symbol CONN_01X01
- added R1: R, symbol R
- added U6: AS7C34098, mod:TSOP44, symbol as7c34098
- U3: footprint (none) -> SMD_Packages:PLCC-32
- gave numbers to parts that had none: 8
Connections:
- net labels added: CLK12, CPUIPL0, CPUIPL1, CPUIPL2, CPULFO, CPURSTI, CPURSTO, CPURW, CPUSCD, CPUSIZ0, CPUSIZ1, CPUTA, CPUTBI, CPUTEA, CPUTIP, CPUTM0, CPUTM1, CPUTM2, CPUTP, CPUTT0, CPUTT1, DAC0CS, DAC1CS, DACWR, LLCE, LLLB, LLOE, LLUB, LLWE, RAM0CS, RAM0LDQM, RAM0UDQM, RAM1CS, RAM1LDQM, RAM1UDQM, RAMA0, RAMA1, RAMA10, RAMA11, RAMA12, RAMA2, RAMA3, RAMA4, RAMA5, RAMA6, RAMA7, RAMA8, RAMA9, RAMB0, RAMB1, RAMCAS, RAMCKE, RAMCLK, RAMRAS, RAMWE, ROMA0, ROMA1, ROMCE, ROMOE, ROMWE, SPICLK, SPIMISO, SPIMOSI, SPISS0, SPISS1, SPISS2, SPISS3, UARTRX, UARTTX, VGAB0, VGAB1, VGAB2, VGAB3, VGAB4, VGAG0, VGAG1, VGAG2, VGAG3, VGAG4, VGAG5, VGAHSYNC, VGAR0, VGAR1, VGAR2, VGAR3, VGAR4, VGAVSYNC
- wire segments 267 -> 371
- no-connect marks 3 -> 14
Other:
- moved on the sheet: U8

Commit message: connectec cpu control signals, spi stuff
Parts:
- removed U3: 39F040, SMD_Packages:PLCC-32, symbol 39F040
- removed U7, U8: TLC7524, Housings_SOIC:SOIC-16_3.9x9.9mm_Pitch1.27mm, symbol TLC7524
- added P?: CONN_01X04, symbol CONN_01X04
- added R? (x3): 1k, symbol R
- added U3: EPC2, Housings_QFP:TQFP-32_7x7mm_Pitch0.8mm, symbol EPC2
- added U7: 74LVC138, Housings_SOIC:SOIC-16_3.9x9.9mm_Pitch1.27mm, symbol 74LS138
- added U8: MCP4902, Housings_SOIC:SOIC-14_3.9x8.7mm_Pitch1.27mm, symbol MCP4922-E/SL
- added U9: S25FL204K0TMFI010, Housings_SOIC:SOIC-8_3.9x4.9mm_Pitch1.27mm, symbol S25FL204K0TMFI010
Connections:
- net labels added: CONF_CLK, CONF_CS, CONF_DATA, CONF_INIT, CONF_OE, EXTINT, SNDSYNC, SPI0CLK, SPI0MISO, SPI0MOSI, SPI0SS1, SPI0SS2, SPI0SS3, SPI0SS4, SPI0SS5, SPI0SS6, SPI0SS7, SPI0SSBIT0, SPI0SSBIT1, SPI0SSBIT2, SPI1CLK, SPI1MOSI, SPI1SS
- net labels removed: DAC0CS, DAC1CS, DACWR, ROMA0, ROMA1, ROMCE, ROMD0, ROMD1, ROMD2, ROMD3, ROMD4, ROMD5, ROMD6, ROMD7, ROMOE, ROMWE, SPICLK, SPIMISO, SPIMOSI, SPISS0, SPISS1, SPISS2, SPISS3
- wire segments 371 -> 502
- no-connect marks 14 -> 17
Other:
- note added: "DAC: MCP4902\nROM: random spi flash"
- note added: "ROM\nTGB\nSD"
- note added: "all these can be user io"
- note added: "more external interrupts?"
- note added: "reset here?"
- note added: "these can be user io"
- moved on the sheet: CON1

Commit message: cpu control signals, vga dac
Parts:
- added P4: ER-CON40HT-1, mod:ER-CON40HT-1, symbol ER-CON40HT-1
- added Q1, Q2: 2N7002E, Housings_SOT-23_SOT-143_TSOT-6:SOT-23_Handsoldering, symbol Q_NMOS_GSD
- added Q3: Q_PMOS_DGS, symbol Q_PMOS_DGS
- added R10, R11, R15: R, symbol R
- added R12: 10k, symbol R
- added R13: 470k, symbol R
- added R14: 20R, symbol R
- added R16, R17, R18: 10k, Resistors_SMD:R_0805_HandSoldering, symbol R
- added R19, R20, R23: 560k, Resistors_SMD:R_0805_HandSoldering, symbol R
- added R21, R22, R24: 180k, Resistors_SMD:R_0805_HandSoldering, symbol R
- added R25, R26, R27: 75, Resistors_SMD:R_0805_HandSoldering, symbol R
- added RP1, RP2, RP3, RP4: 20k, mod:RPACK8_SMD, symbol R_PACK4
- added RP5, RP6, RP7, RP8: 10k, mod:RPACK8_SMD, symbol R_PACK4
- added U10: ADA4851-4, Housings_SSOP:TSSOP-14_4.4x5mm_Pitch0.65mm, symbol ADA4851-4
- CON1: value AVR-JTAG-10 -> FPGA JTAG; footprint AVR-JTAG-10 -> Pin_Headers:Pin_Header_Straight_2x05
- CON2: value AVR-JTAG-10 -> CPU JTAG; footprint AVR-JTAG-10 -> Pin_Headers:Pin_Header_Straight_2x05
- gave numbers to parts that had none: 4
Connections:
- net labels added: EXTINT0, EXTINT1, EXTINT2, EXTINT3, GLOBAL_RESET, VGADEN, VGADISP, VGALED_ANODE, VGALED_CATHODE, VGALED_PWM, VGAPWR
- net labels removed: EXTINT
- wire segments 502 -> 671
- no-connect marks 17 -> 23
Other:
- note added: "Display: ER-TFT070-4"
- note added: "might need backlight pwm here"
- note added: "might need some pullups here somewhere"
- note added: "pixelclock"
- note added: "pull down clken"
- note added: "pull up chip enable"
- note added: "todo: check pinout"
- note added: "user io here too"
- note removed: "more external interrupts?"
- note removed: "reset here?"
- moved on the sheet: CON1

Commit message: almost done
Parts:
- added P5: Power, Pin_Headers:Pin_Header_Straight_1x04, symbol CONN_01X04
- added P6: Peripheral, Pin_Headers:Pin_Header_Straight_1x16, symbol CONN_01X16
- added P7: VGA, Pin_Headers:Pin_Header_Straight_1x06, symbol CONN_01X06
- added P8: Clocks, Pin_Headers:Pin_Header_Straight_1x04, symbol CONN_01X04
- added R28: 1k, Resistors_SMD:R_0805_HandSoldering, symbol R
- added R29: R, Resistors_SMD:R_0805_HandSoldering, symbol R
- added RP10, RP9: R_PACK4, mod:RPACK8_SMD, symbol R_PACK4
- added U11: 33 MHz, trollbook:OSC-VCC1-B3B, symbol VCC1-B3B
- added U12: 12.288 MHz, trollbook:OSC-ASFLMB, symbol VCC1-B3B
- added ZD1: 5V1, symbol ZENER
- P1: value CONN_01X01 -> /BR; footprint (none) -> Measurement_Points:Measurement_Point_Square-SMD-Pad_Small
- P2: value CONN_01X02 -> /CDIS; footprint (none) -> Resistors_SMD:R_0805
- P3: value CONN_01X04 -> Audio; footprint (none) -> Pin_Headers:Pin_Header_Straight_1x04
- Q3: value Q_PMOS_DGS -> DMP3030SN-7; footprint (none) -> Housings_SOT-23_SOT-143_TSOT-6:SOT-23_Handsoldering; symbol Q_PMOS_DGS -> Q_PMOS_GSD
- R1, R10, R11, R12, R13, R14, R15, R2, R3, R4, R5, R6, R7, R8, R9: footprint (none) -> Resistors_SMD:R_0805_HandSoldering
Connections:
- net labels added: CONF_TDO, CPUBB, CPUBG, CPUBR, CPUCDIS, CPUCLK, CPULOC, CPUSC0, CPUSC1, CPUTCK, CPUTDI, CPUTDO, CPUTMS, FPGA_TCK, FPGA_TDI, FPGA_TDO, FPGA_TMS, PWRON_RESET
- net labels removed: GLOBAL_RESET, RAMCLK
- wire segments 671 -> 770
- no-connect marks 23 -> 27
Other:
- note added: "5V sync?"
- note removed: "these can be user io"
- note removed: "user io here too"
- moved on the sheet: CON1, CON2
