File: peripheral-board/power.sch (KiCad schematic (older format))
At the start: 40 parts, among them CON4001 BARREL_JACK, Q4001 Q_PMOS_DGS, Q4002 Q_NMOS_DGS, U4001 AP1509, U4002 LM27313, U4003 LT3652

Commit message: audio circuitry
Parts:
- R4001, R4002, R4003, R4004, R4005, R4006, R4007, R4008, R4009, R4010, R4011, R4012, R4013: footprint (none) -> Resistors_SMD:R_0805
Changed lines of the file:
@@
 EESchema Schematic File Version 2
+LIBS:peripheral-board-rescue
 LIBS:power
 LIBS:device
@@
 LIBS:digital-pot
 LIBS:vref
+LIBS:switches
 LIBS:peripheral-board-cache
 EELAYER 26 0
@@
 $EndComp
 $Comp
-L GND #PWR024
+L GND #PWR4008
 U 1 1 589A1FA0
 P 7400 1650
-F 0 "#PWR024" H -650 -250 50  0001 C CNN
+F 0 "#PWR4008" H -650 -250 50  0001 C CNN
 F 1 "GND" V 7405 1522 50  0000 R CNN
 F 2 "" H -650 0   50  0001 C CNN
@@
 F 0 "R4007" H 6600 2450 50  0000 L CNN
 F 1 "626k" H 6620 2355 50  0000 L CNN
-F 2 "" V -1370 -150 50  0001 C CNN
+F 2 "Resistors_SMD:R_0805" V -1370 -150 50  0001 C CNN
 F 3 "" H -1300 -150 50  0001 C CNN
 	1    6550 2400
@@
 F 0 "R4009" V 7000 2550 50  0000 C CNN
 F 1 "412k" V 6900 2550 50  0000 C CNN
-F 2 "" V -1170 50  50  0001 C CNN
+F 2 "Resistors_SMD:R_0805" V -1170 50  50  0001 C CNN
 F 3 "" H -1100 50  50  0001 C CNN
 	1    6900 2550
@@
 $EndComp
 $Comp
-L GND #PWR025
+L GND #PWR4010
 U 1 1 589A2378
 P 7550 2550
-F 0 "#PWR025" H 7600 2600 50  0001 C CNN
+F 0 "#PWR4010" H 7600 2600 50  0001 C CNN
 F 1 "GND" V 7550 2350 50  0000 C CNN
 F 2 "" H -400 -250 50  0001 C CNN
@@
 F 0 "R4005" V 7200 2050 50  0000 C CNN
 F 1 "0R05" V 7300 2050 50  0000 C CNN
-F 2 "" V -420 -350 50  0001 C CNN
+F 2 "Resistors_SMD:R_0805" V -420 -350 50  0001 C CNN
 F 3 "" H -350 -350 50  0001 C CNN
 	1    7300 2050
@@
 Connection ~ 6950 2250
 $Comp
-L +BATT #PWR026
+L +BATT #PWR4009
 U 1 1 589A3E06
 P 7850 2000
-F 0 "#PWR026" H 0   450 50  0001 C CNN
+F 0 "#PWR4009" H 0   450 50  0001 C CNN
 F 1 "+BATT" H 7865 2173 50  0000 C CNN
 F 2 "" H 0   600 50  0001 C CNN
@@
 Connection ~ 7850 2050
 $Comp
-L GND #PWR027
+L GND #PWR4012
 U 1 1 589A4F62
 P 5650 2950
-F 0 "#PWR027" H -400 -450 50  0001 C CNN
+F 0 "#PWR4012" H -400 -450 50  0001 C CNN
 F 1 "GND" H 5655 2777 50  0000 C CNN
 F 2 "" H -400 -200 50  0001 C CNN
@@
 F 0 "R4003" V 4700 1650 50  0000 C CNN
 F 1 "10k" V 4800 1650 50  0000 C CNN
-F 2 "" V 80  100 50  0001 C CNN
+F 2 "Resistors_SMD:R_0805" V 80  100 50  0001 C CNN
 F 3 "" H 150 100 50  0001 C CNN
 	1    4800 1650
@@
 F 0 "R4004" V 4900 1750 50  0000 C CNN
 F 1 "10k" V 4800 1750 50  0000 C CNN
-F 2 "" V 80  200 50  0001 C CNN
+F 2 "Resistors_SMD:R_0805" V 80  200 50  0001 C CNN
 F 3 "" H 150 200 50  0001 C CNN
 	1    4800 1750
@@
 $EndComp
 $Comp
-L GND #PWR028
+L GND #PWR4007
 U 1 1 589A711D
 P 3650 1550
-F 0 "#PWR028" H 100 -1700 50  0001 C CNN
+F 0 "#PWR4007" H 100 -1700 50  0001 C CNN
 F 1 "GND" H 3655 1377 50  0000 C CNN
 F 2 "" H 100 -1450 50  0001 C CNN
@@
 F 0 "R4006" H 3470 2196 50  0000 L CNN
 F 1 "47k" H 3470 2105 50  0000 L CNN
-F 2 "" V -2270 1050 50  0001 C CNN
+F 2 "Resistors_SMD:R_0805" V -2270 1050 50  0001 C CNN
 F 3 "" H -2200 1050 50  0001 C CNN
 	1    3400 2150
@@
 F 0 "R4002" H 3720 896 50  0000 L CNN
 F 1 "330k" H 3720 805 50  0000 L CNN
-F 2 "" V -2370 50  50  0001 C CNN
+F 2 "Resistors_SMD:R_0805" V -2370 50  50  0001 C CNN
 F 3 "" H -2300 50  50  0001 C CNN
 	1    3650 850
@@
 F 0 "R4008" H 3470 2596 50  0000 L CNN
 F 1 "51k" H 3470 2505 50  0000 L CNN
-F 2 "" V -120 -250 50  0001 C CNN
+F 2 "Resistors_SMD:R_0805" V -120 -250 50  0001 C CNN
 F 3 "" H -50 -250 50  0001 C CNN
 	1    3400 2550
@@
 Connection ~ 3400 2350
 $Comp
-L GND #PWR029
+L GND #PWR4011
 U 1 1 589A7BC3
 P 3400 2700
-F 0 "#PWR029" H -150 -550 50  0001 C CNN
+F 0 "#PWR4011" H -150 -550 50  0001 C CNN
 F 1 "GND" H 3405 2527 50  0000 C CNN
 F 2 "" H -150 -300 50  0001 C CNN
@@
 Connection ~ 3650 650
 $Comp
-L GND #PWR030
+L GND #PWR4006
 U 1 1 589A855C
 P 2200 1450
-F 0 "#PWR030" H -500 -950 50  0001 C CNN
+F 0 "#PWR4006" H -500 -950 50  0001 C CNN
 F 1 "GND" H 2205 1277 50  0000 C CNN
 F 2 "" H -500 -700 50  0001 C CNN
@@
 	2200 1400 2200 1450
 $Comp
-L +12V #PWR031
+L +12V #PWR4002
 U 1 1 589A8BB3
 P 2500 950
-F 0 "#PWR031" H -600 -250 50  0001 C CNN
+F 0 "#PWR4002" H -600 -250 50  0001 C CNN
 F 1 "+12V" H 2515 1123 50  0000 C CNN
 F 2 "" H -600 -100 50  0001 C CNN
@@
 $EndComp
 $Comp
-L PWR_FLAG #FLG032
+L PWR_FLAG #FLG4001
 U 1 1 589A8CB7
 P 2200 950
-F 0 "#FLG032" H -550 -275 50  0001 C CNN
+F 0 "#FLG4001" H -550 -275 50  0001 C CNN
 F 1 "PWR_FLAG" H 2200 1124 50  0000 C CNN
 F 2 "" H -550 -350 50  0001 C CNN
@@
 BATTERY_NTC
 $Comp
-L PWR_FLAG #FLG033
+L PWR_FLAG #FLG4003
 U 1 1 589AA4ED
 P 7500 2000
-F 0 "#FLG033" H 7550 2050 50  0001 C CNN
+F 0 "#FLG4003" H 7550 2050 50  0001 C CNN
 F 1 "PWR_FLAG" H 7500 2174 50  0000 C CNN
 F 2 "" H -550 -1000 50  0001 C CNN
@@
 $EndComp
 $Comp
-L +BATT #PWR034
+L +BATT #PWR4004
 U 1 1 589B38CB
 P 8550 1300
-F 0 "#PWR034" H 700 -250 50  0001 C CNN
+F 0 "#PWR4004" H 700 -250 50  0001 C CNN
 F 1 "+BATT" H 8565 1473 50  0000 C CNN
 F 2 "" H 700 -100 50  0001 C CNN
@@
 $EndComp
 $Comp
-L +12V #PWR035
+L +12V #PWR4003
 U 1 1 589B39F6
 P 8550 1000
-F 0 "#PWR035" H 5450 -200 50  0001 C CNN
+F 0 "#PWR4003" H 5450 -200 50  0001 C CNN
 F 1 "+12V" H 8565 1173 50  0000 C CNN
 F 2 "" H 5450 -50 50  0001 C CNN
@@
 F 0 "R4001" V 9807 750 50  0000 C CNN
 F 1 "10k" V 9716 750 50  0000 C CNN
-F 2 "" V 5130 -2950 50  0001 C CNN
+F 2 "Resistors_SMD:R_0805" V 5130 -2950 50  0001 C CNN
 F 3 "" H 5200 -2950 50  0001 C CNN
 	1    9600 750
@@
 $EndComp
 $Comp
-L GND #PWR036
+L GND #PWR4001
 U 1 1 589B4E54
 P 9450 750
-F 0 "#PWR036" H 6200 -3050 50  0001 C CNN
+F 0 "#PWR4001" H 6200 -3050 50  0001 C CNN
 F 1 "GND" V 9455 622 50  0000 R CNN
 F 2 "" H 6200 -2800 50  0001 C CNN
@@
 	9950 1300 10950 1300
 $Comp
-L VCC #PWR037
+L VCC #PWR4005
 U 1 1 589B6465
 P 10950 1300
-F 0 "#PWR037" H 6250 -3050 50  0001 C CNN
+F 0 "#PWR4005" H 6250 -3050 50  0001 C CNN
 F 1 "VCC" H 10967 1473 50  0000 C CNN
 F 2 "" H 6250 -2900 50  0001 C CNN
@@
 $EndComp
 $Comp
-L PWR_FLAG #FLG038
+L PWR_FLAG #FLG4002
 U 1 1 589B64BF
 P 10700 1300
-F 0 "#FLG038" H 6350 -3025 50  0001 C CNN
+F 0 "#FLG4002" H 6350 -3025 50  0001 C CNN
 F 1 "PWR_FLAG" H 10700 1474 50  0000 C CNN
 F 2 "" H 6350 -3100 50  0001 C CNN
@@
 P 8950 5200
 F 0 "L4003" V 8900 5200 50  0000 C CNN
-F 1 "47u" V 8800 5200 50  0000 C CNN
+F 1 "47u" V 9000 5050 50  0000 C CNN
 F 2 "Choke_SMD:Choke_SMD_7.3x7.3_H4.5" H 100 -200 50  0001 C CNN
 F 3 "" H 100 -200 50  0001 C CNN
@@
 Connection ~ 7900 4600
 $Comp
-L VCC #PWR039
+L VCC #PWR4015
 U 1 1 589B80A7
 P 7900 4400
-F 0 "#PWR039" H 7950 4450 50  0001 C CNN
+F 0 "#PWR4015" H 7950 4450 50  0001 C CNN
 F 1 "VCC" H 7917 4573 50  0000 C CNN
 F 2 "" H 500 0   50  0001 C CNN
@@
 $EndComp
 $Comp
-L GND #PWR040
+L GND #PWR4017
 U 1 1 589B8109
 P 7550 4600
-F 0 "#PWR040" H 7600 4650 50  0001 C CNN
+F 0 "#PWR4017" H 7600 4650 50  0001 C CNN
 F 1 "GND" V 7555 4472 50  0000 R CNN
 F 2 "" H 500 -200 50  0001 C CNN
@@
 Connection ~ 8600 5700
 $Comp
-L GND #PWR041
+L GND #PWR4021
 U 1 1 589B85D2
 P 7750 5750
-F 0 "#PWR041" H 7800 5800 50  0001 C CNN
+F 0 "#PWR4021" H 7800 5800 50  0001 C CNN
 F 1 "GND" H 7755 5577 50  0000 C CNN
 F 2 "" H 650 -750 50  0001 C CNN
@@
 Connection ~ 8600 5200
 $Comp
-L +3V3 #PWR042
+L +3V3 #PWR4019
 U 1 1 589B91D5
 P 9900 5200
-F 0 "#PWR042" H 9950 5250 50  0001 C CNN
+F 0 "#PWR4019" H 9950 5250 50  0001 C CNN
 F 1 "+3V3" H 9915 5373 50  0000 C CNN
 F 2 "" H 1700 -500 50  0001 C CNN
@@
 $EndComp
 $Comp
-L PWR_FLAG #FLG043
+L PWR_FLAG #FLG4005
 U 1 1 589B9237
 P 9450 5200
-F 0 "#FLG043" H 9500 5250 50  0001 C CNN
+F 0 "#FLG4005" H 9500 5250 50  0001 C CNN
 F 1 "PWR_FLAG" H 9450 5374 50  0000 C CNN
 F 2 "" H 1200 -550 50  0001 C CNN
@@
 $EndComp
 $Comp
-L VCC #PWR044
+L VCC #PWR4014
 U 1 1 589BA1AA
 P 3000 4400
-F 0 "#PWR044" H 3050 4450 50  0001 C CNN
+F 0 "#PWR4014" H 3050 4450 50  0001 C CNN
 F 1 "VCC" H 3017 4573 50  0000 C CNN
 F 2 "" H -4400 0   50  0001 C CNN
@@
 	3000 4400 3000 4500
 $Comp
-L GND #PWR045
+L GND #PWR4016
 U 1 1 589BA9B7
 P 2650 4450
-F 0 "#PWR045" H 2700 4500 50  0001 C CNN
+F 0 "#PWR4016" H 2700 4500 50  0001 C CNN
 F 1 "GND" V 2655 4322 50  0000 R CNN
 F 2 "" H -4450 -2050 50  0001 C CNN
@@
 $EndComp
 $Comp
-L GND #PWR046
+L GND #PWR4020
 U 1 1 589BAA61
 P 3000 5750
-F 0 "#PWR046" H 3050 5800 50  0001 C CNN
+F 0 "#PWR4020" H 3050 5800 50  0001 C CNN
 F 1 "GND" H 3005 5577 50  0000 C CNN
 F 2 "" H -4100 -750 50  0001 C CNN
@@
 F 0 "R4012" V 3850 4950 50  0000 C CNN
 F 1 "270k" V 3950 5100 50  0000 C CNN
-F 2 "" V -1070 -400 50  0001 C CNN
+F 2 "Resistors_SMD:R_0805" V -1070 -400 50  0001 C CNN
 F 3 "" H -1000 -400 50  0001 C CNN
 	1    3950 5100
@@
 F 0 "R4013" H 3820 5596 50  0000 L CNN
 F 1 "13.3k" H 3820 5505 50  0000 L CNN
-F 2 "" V -1420 -200 50  0001 C CNN
+F 2 "Resistors_SMD:R_0805" V -1420 -200 50  0001 C CNN
 F 3 "" H -1350 -200 50  0001 C CNN
 	1    3750 5550
@@
 Connection ~ 3750 5300
 $Comp
-L +24V #PWR047
+L +24V #PWR4018
 U 1 1 589BBC33
 P 4800 5000
-F 0 "#PWR047" H 4850 5050 50  0001 C CNN
+F 0 "#PWR4018" H 4850 5050 50  0001 C CNN
 F 1 "+24V" H 4815 5173 50  0000 C CNN
 F 2 "" H -100 -50 50  0001 C CNN
@@
 $EndComp
 $Comp
-L PWR_FLAG #FLG048
+L PWR_FLAG #FLG4004
 U 1 1 589BBD5B
 P 4500 5000
-F 0 "#FLG048" H 4550 5050 50  0001 C CNN
+F 0 "#FLG4004" H 4550 5050 50  0001 C CNN
 F 1 "PWR_FLAG" H 4500 5174 50  0000 C CNN
 F 2 "" H -400 -550 50  0001 C CNN
@@
 F 0 "R4011" H 2170 4896 50  0000 L CNN
 F 1 "R" H 2170 4805 50  0000 L CNN
-F 2 "" V -120 -50 50  0001 C CNN
+F 2 "Resistors_SMD:R_0805" V -120 -50 50  0001 C CNN
 F 3 "" H -50 -50 50  0001 C CNN
 	1    2100 4850
@@
 F 0 "R4010" H 1220 4096 50  0000 L CNN
 F 1 "R" H 1220 4005 50  0000 L CNN
-F 2 "" V 30  -250 50  0001 C CNN
+F 2 "Resistors_SMD:R_0805" V 30  -250 50  0001 C CNN
 F 3 "" H 100 -250 50  0001 C CNN
 	1    1150 4050
@@
 $EndComp
 $Comp
-L GND #PWR049
+L GND #PWR4013
 U 1 1 589BF9D9
 P 1150 4250
-F 0 "#PWR049" H 200 -500 50  0001 C CNN
+F 0 "#PWR4013" H 200 -500 50  0001 C CNN
 F 1 "GND" H 1155 4077 50  0000 C CNN
 F 2 "" H 200 -250 50  0001 C CNN
