File: peripheral-board/rtc.sch (KiCad schematic (older format))
At the start: 4 parts, among them U5001 MCP7940N, Y5001 32768 Hz

Commit message: routed traces.
Parts:
- C5001, C5002: value C_Small -> 22p
Connections:
- net +3.3VP: now reaches U5001.3 (VBAT)
Changed lines of the file:
@@
 P 6250 3200
 F 0 "C5001" V 6021 3200 50  0000 C CNN
-F 1 "C_Small" V 6112 3200 50  0000 C CNN
+F 1 "22p" V 6112 3200 50  0000 C CNN
 F 2 "Capacitors_SMD:C_0603" H 6250 3200 50  0001 C CNN
 F 3 "" H 6250 3200 50  0000 C CNN
@@
 P 6250 3600
 F 0 "C5002" V 6500 3600 50  0000 C CNN
-F 1 "C_Small" V 6400 3600 50  0000 C CNN
+F 1 "22p" V 6400 3600 50  0000 C CNN
 F 2 "Capacitors_SMD:C_0603" H 6250 3600 50  0001 C CNN
 F 3 "" H 6250 3600 50  0000 C CNN
@@
 	6150 3500 6150 3600
 $Comp
-L GND #PWR057
+L GND #PWR060
 U 1 1 58221B92
 P 6400 3200
-F 0 "#PWR057" H 6400 2950 50  0001 C CNN
+F 0 "#PWR060" H 6400 2950 50  0001 C CNN
 F 1 "GND" V 6405 3072 50  0000 R CNN
 F 2 "" H 6400 3200 50  0000 C CNN
@@
 $EndComp
 $Comp
-L GND #PWR058
+L GND #PWR061
 U 1 1 58221BBA
 P 6400 3600
-F 0 "#PWR058" H 6400 3350 50  0001 C CNN
+F 0 "#PWR061" H 6400 3350 50  0001 C CNN
 F 1 "GND" V 6405 3472 50  0000 R CNN
 F 2 "" H 6400 3600 50  0000 C CNN
@@
 NoConn ~ 5200 3500
 $Comp
-L GND #PWR059
+L GND #PWR062
 U 1 1 58221C3E
-P 5600 3850
-F 0 "#PWR059" H 5600 3600 50  0001 C CNN
-F 1 "GND" H 5605 3677 50  0000 C CNN
-F 2 "" H 5600 3850 50  0000 C CNN
-F 3 "" H 5600 3850 50  0000 C CNN
-	1    5600 3850
+P 5600 3800
+F 0 "#PWR062" H 5600 3550 50  0001 C CNN
+F 1 "GND" H 5605 3627 50  0000 C CNN
+F 2 "" H 5600 3800 50  0000 C CNN
+F 3 "" H 5600 3800 50  0000 C CNN
+	1    5600 3800
 	1    0    0    -1
 $EndComp
 $Comp
-L +3V3 #PWR060
+L +3V3 #PWR063
 U 1 1 58221C5A
-P 5600 2950
-F 0 "#PWR060" H 5600 2800 50  0001 C CNN
-F 1 "+3V3" H 5615 3123 50  0000 C CNN
-F 2 "" H 5600 2950 50  0000 C CNN
-F 3 "" H 5600 2950 50  0000 C CNN
-	1    5600 2950
+P 5600 3000
+F 0 "#PWR063" H 5600 2850 50  0001 C CNN
+F 1 "+3V3" H 5450 3100 50  0000 C CNN
+F 2 "" H 5600 3000 50  0000 C CNN
+F 3 "" H 5600 3000 50  0000 C CNN
+	1    5600 3000
 	1    0    0    -1
 $EndComp
-Wire Wire Line
-	5600 2950 5600 3000
-Wire Wire Line
-	5600 3800 5600 3850
 Text HLabel 4800 3200 0    60   Input ~ 0
 SCL
@@
 Wire Wire Line
 	5200 3300 4800 3300
+$Comp
+L +3.3VP #PWR064
+U 1 1 58A61230
+P 5700 3000
+F 0 "#PWR064" H -50 250 50  0001 C CNN
+F 1 "+3.3VP" H 5850 3100 50  0000 C CNN
+F 2 "" H -200 300 50  0001 C CNN
+F 3 "" H -200 300 50  0001 C CNN
+	1    5700 3000
+	1    0    0    -1
+$EndComp
 $EndSCHEMATC
