File: peripheral-board/audio.sch (KiCad schematic (older format))
At the start: 31 parts, among them J7001 FCR1295, U7001 LM386, U7002 LM386, U7003 MCP4011, U7004 MCP4011

Commit message: routed traces.
Parts:
- C7007, C7014: footprint Capacitors_SMD:C_0805 -> Capacitors_SMD:C_1206
Changed lines of the file:
@@
 $EndComp
 $Comp
-L GND #PWR061
+L GND #PWR065
 U 1 1 5823647F
 P 3300 3450
-F 0 "#PWR061" H 3300 3200 50  0001 C CNN
+F 0 "#PWR065" H 3300 3200 50  0001 C CNN
 F 1 "GND" H 3305 3277 50  0000 C CNN
 F 2 "" H 3300 3450 50  0000 C CNN
@@
 $EndComp
 $Comp
-L GND #PWR062
+L GND #PWR066
 U 1 1 582364AF
 P 3300 4850
-F 0 "#PWR062" H 3300 4600 50  0001 C CNN
+F 0 "#PWR066" H 3300 4600 50  0001 C CNN
 F 1 "GND" H 3305 4677 50  0000 C CNN
 F 2 "" H 3300 4850 50  0000 C CNN
@@
 $EndComp
 $Comp
-L +3V3 #PWR063
+L +3V3 #PWR067
 U 1 1 582364E9
 P 3300 2350
-F 0 "#PWR063" H 3300 2200 50  0001 C CNN
+F 0 "#PWR067" H 3300 2200 50  0001 C CNN
 F 1 "+3V3" V 3315 2478 50  0000 L CNN
 F 2 "" H 3300 2350 50  0000 C CNN
@@
 $EndComp
 $Comp
-L +3V3 #PWR064
+L +3V3 #PWR068
 U 1 1 58236543
 P 3350 3800
-F 0 "#PWR064" H 3350 3650 50  0001 C CNN
+F 0 "#PWR068" H 3350 3650 50  0001 C CNN
 F 1 "+3V3" V 3365 3928 50  0000 L CNN
 F 2 "" H 3350 3800 50  0000 C CNN
@@
 DETECT
 $Comp
-L GND #PWR065
+L GND #PWR069
 U 1 1 58240DA5
 P 4100 3300
-F 0 "#PWR065" H 4100 3050 50  0001 C CNN
+F 0 "#PWR069" H 4100 3050 50  0001 C CNN
 F 1 "GND" H 4105 3127 50  0000 C CNN
 F 2 "" H 4100 3300 50  0000 C CNN
@@
 $EndComp
 $Comp
-L GND #PWR066
+L GND #PWR070
 U 1 1 58A1A8BA
 P 10050 3400
-F 0 "#PWR066" H 10100 3450 50  0001 C CNN
+F 0 "#PWR070" H 10100 3450 50  0001 C CNN
 F 1 "GND" V 10055 3272 50  0000 R CNN
 F 2 "" H 1200 200 50  0001 C CNN
@@
 $EndComp
 $Comp
-L +3V3 #PWR067
+L +3V3 #PWR071
 U 1 1 58A1A914
 P 9950 3000
-F 0 "#PWR067" H 10000 3050 50  0001 C CNN
+F 0 "#PWR071" H 10000 3050 50  0001 C CNN
 F 1 "+3V3" V 9965 3128 50  0000 L CNN
 F 2 "" H 1550 -100 50  0001 C CNN
@@
 $EndComp
 $Comp
-L GND #PWR068
+L GND #PWR072
 U 1 1 58A1ACEA
 P 10000 4500
-F 0 "#PWR068" H 10050 4550 50  0001 C CNN
+F 0 "#PWR072" H 10050 4550 50  0001 C CNN
 F 1 "GND" V 10005 4372 50  0000 R CNN
 F 2 "" H 600 1650 50  0001 C CNN
@@
 $EndComp
 $Comp
-L GND #PWR069
+L GND #PWR073
 U 1 1 58A1AD9C
 P 10000 2650
-F 0 "#PWR069" H 10050 2700 50  0001 C CNN
+F 0 "#PWR073" H 10050 2700 50  0001 C CNN
 F 1 "GND" V 10005 2522 50  0000 R CNN
 F 2 "" H 1550 300 50  0001 C CNN
@@
 F 0 "C7007" H 3985 2604 50  0000 R CNN
 F 1 "1u" H 3985 2695 50  0000 R CNN
-F 2 "Capacitors_SMD:C_0805" H -912 -350 50  0001 C CNN
+F 2 "Capacitors_SMD:C_1206" H -912 -350 50  0001 C CNN
 F 3 "" H -950 -200 50  0001 C CNN
 	1    4100 2650
@@
 NoConn ~ 6350 3200
 $Comp
-L GND #PWR070
+L GND #PWR074
 U 1 1 58A359F1
 P 6650 2600
-F 0 "#PWR070" H -400 -250 50  0001 C CNN
+F 0 "#PWR074" H -400 -250 50  0001 C CNN
 F 1 "GND" V 6655 2472 50  0000 R CNN
 F 2 "" H -400 0   50  0001 C CNN
@@
 $EndComp
 $Comp
-L GND #PWR071
+L GND #PWR075
 U 1 1 58A36C12
 P 5750 2600
-F 0 "#PWR071" H -1400 250 50  0001 C CNN
+F 0 "#PWR075" H -1400 250 50  0001 C CNN
 F 1 "GND" V 5755 2472 50  0000 R CNN
 F 2 "" H -1400 500 50  0001 C CNN
@@
 	6250 2250 6250 2600
 $Comp
-L GND #PWR072
+L GND #PWR076
 U 1 1 58A3787F
 P 4100 4700
-F 0 "#PWR072" H 4100 4450 50  0001 C CNN
+F 0 "#PWR076" H 4100 4450 50  0001 C CNN
 F 1 "GND" H 4105 4527 50  0000 C CNN
 F 2 "" H 4100 4700 50  0000 C CNN
@@
 F 0 "C7014" H 3985 4004 50  0000 R CNN
 F 1 "1u" H 3985 4095 50  0000 R CNN
-F 2 "Capacitors_SMD:C_0805" H -912 1050 50  0001 C CNN
+F 2 "Capacitors_SMD:C_1206" H -912 1050 50  0001 C CNN
 F 3 "" H -950 1200 50  0001 C CNN
 	1    4100 4050
@@
 NoConn ~ 6350 4600
 $Comp
-L GND #PWR073
+L GND #PWR077
 U 1 1 58A378BA
 P 6650 4000
-F 0 "#PWR073" H -400 1150 50  0001 C CNN
+F 0 "#PWR077" H -400 1150 50  0001 C CNN
 F 1 "GND" V 6655 3872 50  0000 R CNN
 F 2 "" H -400 1400 50  0001 C CNN
@@
 $EndComp
 $Comp
-L GND #PWR074
+L GND #PWR078
 U 1 1 58A39053
 P 5750 4000
-F 0 "#PWR074" H -1400 1650 50  0001 C CNN
+F 0 "#PWR078" H -1400 1650 50  0001 C CNN
 F 1 "GND" V 5755 3872 50  0000 R CNN
 F 2 "" H -1400 1900 50  0001 C CNN
@@
 $EndComp
 $Comp
-L GND #PWR075
+L GND #PWR079
 U 1 1 58A3B2B9
 P 3000 2350
-F 0 "#PWR075" H 50  -50 50  0001 C CNN
+F 0 "#PWR079" H 50  -50 50  0001 C CNN
 F 1 "GND" V 3005 2222 50  0000 R CNN
 F 2 "" H 50  200 50  0001 C CNN
@@
 $EndComp
 $Comp
-L GND #PWR076
+L GND #PWR080
 U 1 1 58A3B4D5
 P 3000 3800
-F 0 "#PWR076" H 50  1400 50  0001 C CNN
+F 0 "#PWR080" H 50  1400 50  0001 C CNN
 F 1 "GND" V 3005 3672 50  0000 R CNN
 F 2 "" H 50  1650 50  0001 C CNN
@@
 $EndComp
 $Comp
-L VAA #PWR077
+L VAA #PWR081
 U 1 1 58A8FF55
 P 6250 2250
-F 0 "#PWR077" H -2150 900 50  0001 C CNN
+F 0 "#PWR081" H -2150 900 50  0001 C CNN
 F 1 "VAA" H 6267 2423 50  0000 C CNN
 F 2 "" H -2150 1050 50  0001 C CNN
@@
 $EndComp
 $Comp
-L VAA #PWR078
+L VAA #PWR082
 U 1 1 58A9009E
 P 6250 3650
-F 0 "#PWR078" H -2150 2300 50  0001 C CNN
+F 0 "#PWR082" H -2150 2300 50  0001 C CNN
 F 1 "VAA" H 6267 3823 50  0000 C CNN
 F 2 "" H -2150 2450 50  0001 C CNN
@@
 $EndComp
 $Comp
-L VAA #PWR079
+L VAA #PWR083
 U 1 1 58A4CF7D
 P 5100 1800
-F 0 "#PWR079" H -3300 450 50  0001 C CNN
+F 0 "#PWR083" H -3300 450 50  0001 C CNN
 F 1 "VAA" H 5117 1973 50  0000 C CNN
 F 2 "" H -3300 600 50  0001 C CNN
@@
 $EndComp
 $Comp
-L GND #PWR080
+L GND #PWR084
 U 1 1 58A4D14E
 P 5100 2100
-F 0 "#PWR080" H 5100 1850 50  0001 C CNN
+F 0 "#PWR084" H 5100 1850 50  0001 C CNN
 F 1 "GND" H 5105 1927 50  0000 C CNN
 F 2 "" H 5100 2100 50  0000 C CNN
