File: peripheral-board/audio.sch (KiCad schematic (older format))
At the start: 31 parts, among them J7001 FCR1295, U7001 LM386, U7002 LM386, U7003 MCP4011, U7004 MCP4011

Commit message: added speaker and battery connectors
Parts:
- removed LS7001: Speaker L, Socket_Strips:Socket_Strip_Straight_1x02_Pitch2.54mm, symbol Speaker
- removed LS7002: Speaker R, Socket_Strips:Socket_Strip_Straight_1x02_Pitch2.54mm, symbol Speaker
- added J7002: 53047-0310, Connectors_Molex:Connector_Molex_PicoBlade_53047-0410, symbol CONN_01X04_MALE
Connections:
- net GND: now also J7002.1, J7002.3
- net SPKR_L: now also J7002.4
- net SPKR_R: now also J7002.2
Changed lines of the file:
@@
-$EndComp
-$Comp
-L Speaker LS7001
-U 1 1 58A1A3A1
-P 10200 2750
-F 0 "LS7001" H 10164 2333 50  0000 C CNN
-F 1 "Speaker L" H 10164 2424 50  0000 C CNN
-F 2 "Socket_Strips:Socket_Strip_Straight_1x02_Pitch2.54mm" H 1700 1600 50  0001 C CNN
-F 3 "" H 1690 1750 50  0001 C CNN
-	1    10200 2750
-	1    0    0    1
-$EndComp
-$Comp
-L Speaker LS7002
-U 1 1 58A1A483
-P 10200 4400
-F 0 "LS7002" H 10370 4396 50  0000 L CNN
-F 1 "Speaker R" H 10370 4305 50  0000 L CNN
-F 2 "Socket_Strips:Socket_Strip_Straight_1x02_Pitch2.54mm" H 1700 3250 50  0001 C CNN
-F 3 "" H 1690 3400 50  0001 C CNN
-	1    10200 4400
-	1    0    0    -1
 $EndComp
 $Comp
@@
 $EndComp
 $Comp
-L GND #PWR075
-U 1 1 58A1ACEA
-P 10000 4500
-F 0 "#PWR075" H 10050 4550 50  0001 C CNN
-F 1 "GND" V 10005 4372 50  0000 R CNN
-F 2 "" H 600 1650 50  0001 C CNN
-F 3 "" H 600 1650 50  0001 C CNN
-	1    10000 4500
-	0    1    1    0
-$EndComp
-$Comp
-L GND #PWR076
-U 1 1 58A1AD9C
-P 10000 2650
-F 0 "#PWR076" H 10050 2700 50  0001 C CNN
-F 1 "GND" V 10005 2522 50  0000 R CNN
-F 2 "" H 1550 300 50  0001 C CNN
-F 3 "" H 1550 300 50  0001 C CNN
-	1    10000 2650
-	0    1    1    0
-$EndComp
-$Comp
 L LM386 U7001
 U 1 1 58A34689
@@
 	1    0    0    -1
 $EndComp
-Wire Wire Line
-	1700 2850 2550 2850
-Wire Wire Line
-	1800 2950 2550 2950
-Wire Wire Line
-	1700 4250 2550 4250
-Wire Wire Line
-	2550 4350 1900 4350
-Wire Wire Line
-	1700 2850 1700 4550
-Wire Wire Line
-	1700 4550 1600 4550
-Connection ~ 1700 4250
-Wire Wire Line
-	1800 2950 1800 4650
-Wire Wire Line
-	1800 4650 1600 4650
-Wire Wire Line
-	1900 4350 1900 4750
-Wire Wire Line
-	1900 4750 1600 4750
-Wire Wire Line
-	3300 2350 3300 2400
-Wire Wire Line
-	3300 3400 3300 3450
-Wire Wire Line
-	3300 3800 3350 3800
-Wire Wire Line
-	3300 4800 3300 4850
-Wire Wire Line
-	9750 3300 10050 3300
-Wire Wire Line
-	4100 2800 4050 2800
-Wire Wire Line
-	4050 3000 4100 3000
-Wire Wire Line
-	4100 3000 4100 3300
-Wire Wire Line
-	9300 2750 10000 2750
-Wire Wire Line
-	9300 2750 9300 3500
-Wire Wire Line
-	9300 3500 10050 3500
-Connection ~ 9950 3300
-Wire Wire Line
-	10000 4400 9300 4400
-Wire Wire Line
-	9300 4400 9300 3700
-Wire Wire Line
-	9300 3700 10050 3700
-Wire Wire Line
-	4650 2900 5250 2900
-Connection ~ 4950 2900
-Wire Wire Line
-	4350 2900 4050 2900
-Wire Wire Line
-	5250 2900 5250 2800
-Wire Wire Line
-	5250 2800 6050 2800
-Connection ~ 5250 2900
 $Comp
 L C C7006
@@
 	0    -1   -1   0
 $EndComp
-Wire Wire Line
-	6650 2900 7250 2900
-Connection ~ 6950 2900
-Wire Wire Line
-	4100 3300 6650 3300
-Wire Wire Line
-	6250 3300 6250 3200
-Connection ~ 6250 3300
-Wire Wire Line
-	4950 3200 4950 3300
-Connection ~ 4950 3300
-Wire Wire Line
-	5250 3200 5250 3300
-Connection ~ 5250 3300
-Wire Wire Line
-	6050 3000 6050 3300
-Connection ~ 6050 3300
-Wire Wire Line
-	6950 3300 6950 3200
 $Comp
 L C C7005
@@
 	0    1    1    0
 $EndComp
-Wire Wire Line
-	6250 2250 6250 2600
 $Comp
 L GND #PWR079
@@
 	1    0    0    -1
 $EndComp
-Wire Wire Line
-	4100 4200 4050 4200
-Wire Wire Line
-	4050 4400 4100 4400
-Wire Wire Line
-	4100 4400 4100 4700
-Wire Wire Line
-	4650 4300 5250 4300
-Connection ~ 4950 4300
-Wire Wire Line
-	4350 4300 4050 4300
-Wire Wire Line
-	5250 4300 5250 4200
-Wire Wire Line
-	5250 4200 6050 4200
-Connection ~ 5250 4300
 $Comp
 L C C7013
@@
 	0    -1   -1   0
 $EndComp
-Wire Wire Line
-	6650 4300 7250 4300
-Connection ~ 6950 4300
-Wire Wire Line
-	4100 4700 6650 4700
-Wire Wire Line
-	6250 4700 6250 4600
-Connection ~ 6250 4700
-Wire Wire Line
-	4950 4600 4950 4700
-Connection ~ 4950 4700
-Wire Wire Line
-	5250 4600 5250 4700
-Connection ~ 5250 4700
-Wire Wire Line
-	6050 4400 6050 4700
-Connection ~ 6050 4700
-Wire Wire Line
-	6950 4700 6950 4600
-Wire Wire Line
-	10050 3600 8050 3600
-Wire Wire Line
-	8050 3600 8050 2900
-Wire Wire Line
-	8050 2900 7550 2900
-Wire Wire Line
-	10050 3800 8050 3800
-Wire Wire Line
-	8050 3800 8050 4300
-Wire Wire Line
-	8050 4300 7550 4300
 Text Label 8350 3600 0    60   ~ 0
 JACK_L
 Text Label 8350 3800 0    60   ~ 0
 JACK_R
-Text Label 9350 2750 0    60   ~ 0
+Text Label 9350 3500 0    60   ~ 0
 SPKR_L
-Text Label 9350 4400 0    60   ~ 0
+Text Label 9350 3700 0    60   ~ 0
 SPKR_R
 $Comp
@@
 	1    0    0    -1
 $EndComp
-Wire Wire Line
-	5950 2400 5750 2400
-Wire Wire Line
-	5750 2400 5750 2600
-Wire Wire Line
-	5750 2600 5950 2600
-Connection ~ 6250 2400
 $Comp
 L C C7012
@@
 	0    1    1    0
 $EndComp
-Wire Wire Line
-	6250 3650 6250 4000
-Wire Wire Line
-	5950 3800 5750 3800
-Wire Wire Line
-	5750 3800 5750 4000
-Connection ~ 6250 3800
-Wire Wire Line
-	5750 4000 5950 4000
 $Comp
 L C C7001
@@
 	1    0    0    -1
 $EndComp
+$Comp
+L CONN_01X04_MALE J7002
+U 1 1 58AB56D2
+P 9000 1850
+F 0 "J7002" V 9060 1463 50  0000 R CNN
+F 1 "53047-0310" V 9151 1463 50  0000 R CNN
+F 2 "Connectors_Molex:Connector_Molex_PicoBlade_53047-0410" H -1150 200 50  0001 C CNN
+F 3 "" H -1150 200 50  0001 C CNN
+	1    9000 1850
+	0    -1   1    0
+$EndComp
+$Comp
+L GND #PWR088
+U 1 1 58AB598A
+P 8700 2150
+F 0 "#PWR088" H 8750 2200 50  0001 C CNN
+F 1 "GND" H 8705 1977 50  0000 C CNN
+F 2 "" H -1150 150 50  0001 C CNN
+F 3 "" H -1150 150 50  0001 C CNN
+	1    8700 2150
+	1    0    0    -1
+$EndComp
+Wire Wire Line
+	1700 2850 2550 2850
+Wire Wire Line
+	1800 2950 2550 2950
+Wire Wire Line
+	1700 4250 2550 4250
+Wire Wire Line
+	2550 4350 1900 4350
+Wire Wire Line
+	1700 2850 1700 4550
+Wire Wire Line
+	1700 4550 1600 4550
+Connection ~ 1700 4250
+Wire Wire Line
+	1800 2950 1800 4650
+Wire Wire Line
+	1800 4650 1600 4650
+Wire Wire Line
+	1900 4350 1900 4750
+Wire Wire Line
+	1900 4750 1600 4750
+Wire Wire Line
+	3300 2350 3300 2400
+Wire Wire Line
+	3300 3400 3300 3450
+Wire Wire Line
+	3300 3800 3350 3800
+Wire Wire Line
+	3300 4800 3300 4850
+Wire Wire Line
+	9750 3300 10050 3300
+Wire Wire Line
+	4100 2800 4050 2800
+Wire Wire Line
+	4050 3000 4100 3000
+Wire Wire Line
+	4100 3000 4100 3300
+Wire Wire Line
+	9300 2150 9300 3500
+Wire Wire Line
+	9300 3500 10050 3500
+Connection ~ 9950 3300
+Wire Wire Line
+	8900 3700 10050 3700
+Wire Wire Line
+	4650 2900 5250 2900
+Connection ~ 4950 2900
+Wire Wire Line
+	4350 2900 4050 2900
+Wire Wire Line
+	5250 2900 5250 2800
+Wire Wire Line
+	5250 2800 6050 2800
+Connection ~ 5250 2900
+Wire Wire Line
+	6650 2900 7250 2900
+Connection ~ 6950 2900
+Wire Wire Line
+	4100 3300 6650 3300
+Wire Wire Line
+	6250 3300 6250 3200
+Connection ~ 6250 3300
+Wire Wire Line
+	4950 3200 4950 3300
+Connection ~ 4950 3300
+Wire Wire Line
+	5250 3200 5250 3300
+Connection ~ 5250 3300
+Wire Wire Line
+	6050 3000 6050 3300
+Connection ~ 6050 3300
+Wire Wire Line
+	6950 3300 6950 3200
+Wire Wire Line
+	6250 2250 6250 2600
+Wire Wire Line
+	4100 4200 4050 4200
+Wire Wire Line
+	4050 4400 4100 4400
+Wire Wire Line
+	4100 4400 4100 4700
+Wire Wire Line
+	4650 4300 5250 4300
+Connection ~ 4950 4300
+Wire Wire Line
+	4350 4300 4050 4300
+Wire Wire Line
+	5250 4300 5250 4200
+Wire Wire Line
+	5250 4200 6050 4200
+Connection ~ 5250 4300
+Wire Wire Line
+	6650 4300 7250 4300
+Connection ~ 6950 4300
+Wire Wire Line
+	4100 4700 6650 4700
+Wire Wire Line
+	6250 4700 6250 4600
+Connection ~ 6250 4700
+Wire Wire Line
+	4950 4600 4950 4700
+Connection ~ 4950 4700
+Wire Wire Line
+	5250 4600 5250 4700
+Connection ~ 5250 4700
+Wire Wire Line
+	6050 4400 6050 4700
+Connection ~ 6050 4700
+Wire Wire Line
+	6950 4700 6950 4600
+Wire Wire Line
+	10050 3600 8050 3600
+Wire Wire Line
+	8050 3600 8050 2900
+Wire Wire Line
+	8050 2900 7550 2900
+Wire Wire Line
+	10050 3800 8050 3800
+Wire Wire Line
+	8050 3800 8050 4300
+Wire Wire Line
+	8050 4300 7550 4300
+Wire Wire Line
+	5950 2400 5750 2400
+Wire Wire Line
+	5750 2400 5750 2600
+Wire Wire Line
+	5750 2600 5950 2600
+Connection ~ 6250 2400
+Wire Wire Line
+	6250 3650 6250 4000
+Wire Wire Line
+	5950 3800 5750 3800
+Wire Wire Line
+	5750 3800 5750 4000
+Connection ~ 6250 3800
+Wire Wire Line
+	5750 4000 5950 4000
+Wire Wire Line
+	8900 3700 8900 2150
+$Comp
+L GND #PWR089
+U 1 1 58AB708B
+P 9100 2150
+F 0 "#PWR089" H 9150 2200 50  0001 C CNN
+F 1 "GND" H 9105 1977 50  0000 C CNN
+F 2 "" H -750 150 50  0001 C CNN
+F 3 "" H -750 150 50  0001 C CNN
+	1    9100 2150
+	1    0    0    -1
+$EndComp

Commit message: minor fixes to peripheral board
Parts:
- added R6001, R6002: 10k, Resistors_SMD:R_0805, symbol R
Connections:
- net +3V3: now also R6001.1, R6002.1
- net at C7009.1, R7003.1, R7004.1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: now also R6001.2
- net at C7016.1, R7007.1, R7008.1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: now also R6002.2
Changed lines of the file:
@@
 $Descr A4 11693 8268
 encoding utf-8
-Sheet 7 8
+Sheet 6 8
 Title ""
 Date ""
@@
 $EndComp
 $Comp
-L GND #PWR068
+L GND #PWR6014
 U 1 1 5823647F
 P 3300 3450
-F 0 "#PWR068" H 3300 3200 50  0001 C CNN
+F 0 "#PWR6014" H 3300 3200 50  0001 C CNN
 F 1 "GND" H 3305 3277 50  0000 C CNN
 F 2 "" H 3300 3450 50  0000 C CNN
@@
 $EndComp
 $Comp
-L GND #PWR069
+L GND #PWR6022
 U 1 1 582364AF
 P 3300 4850
-F 0 "#PWR069" H 3300 4600 50  0001 C CNN
+F 0 "#PWR6022" H 3300 4600 50  0001 C CNN
 F 1 "GND" H 3305 4677 50  0000 C CNN
 F 2 "" H 3300 4850 50  0000 C CNN
@@
 $EndComp
 $Comp
-L +3V3 #PWR070
+L +3V3 #PWR6007
 U 1 1 582364E9
 P 3300 2350
-F 0 "#PWR070" H 3300 2200 50  0001 C CNN
+F 0 "#PWR6007" H 3300 2200 50  0001 C CNN
 F 1 "+3V3" V 3315 2478 50  0000 L CNN
 F 2 "" H 3300 2350 50  0000 C CNN
@@
 $EndComp
 $Comp
-L +3V3 #PWR071
+L +3V3 #PWR6017
 U 1 1 58236543
 P 3350 3800
-F 0 "#PWR071" H 3350 3650 50  0001 C CNN
+F 0 "#PWR6017" H 3350 3650 50  0001 C CNN
 F 1 "+3V3" V 3365 3928 50  0000 L CNN
 F 2 "" H 3350 3800 50  0000 C CNN
@@
 DETECT
 $Comp
-L GND #PWR072
+L GND #PWR6012
 U 1 1 58240DA5
 P 4100 3300
-F 0 "#PWR072" H 4100 3050 50  0001 C CNN
+F 0 "#PWR6012" H 4100 3050 50  0001 C CNN
 F 1 "GND" H 4105 3127 50  0000 C CNN
 F 2 "" H 4100 3300 50  0000 C CNN
@@
 $EndComp
 $Comp
-L GND #PWR073
+L GND #PWR6013
 U 1 1 58A1A8BA
 P 10050 3400
-F 0 "#PWR073" H 10100 3450 50  0001 C CNN
+F 0 "#PWR6013" H 10100 3450 50  0001 C CNN
 F 1 "GND" V 10055 3272 50  0000 R CNN
 F 2 "" H 1200 200 50  0001 C CNN
@@
 $EndComp
 $Comp
-L +3V3 #PWR074
+L +3V3 #PWR6011
 U 1 1 58A1A914
 P 9950 3000
-F 0 "#PWR074" H 10000 3050 50  0001 C CNN
+F 0 "#PWR6011" H 10000 3050 50  0001 C CNN
 F 1 "+3V3" V 9965 3128 50  0000 L CNN
 F 2 "" H 1550 -100 50  0001 C CNN
@@
 NoConn ~ 6350 3200
 $Comp
-L GND #PWR075
+L GND #PWR6010
 U 1 1 58A359F1
 P 6650 2600
-F 0 "#PWR075" H -400 -250 50  0001 C CNN
+F 0 "#PWR6010" H -400 -250 50  0001 C CNN
 F 1 "GND" V 6655 2472 50  0000 R CNN
 F 2 "" H -400 0   50  0001 C CNN
@@
 $EndComp
 $Comp
-L GND #PWR076
+L GND #PWR6009
 U 1 1 58A36C12
 P 5750 2600
-F 0 "#PWR076" H -1400 250 50  0001 C CNN
+F 0 "#PWR6009" H -1400 250 50  0001 C CNN
 F 1 "GND" V 5755 2472 50  0000 R CNN
 F 2 "" H -1400 500 50  0001 C CNN
@@
 $EndComp
 $Comp
-L GND #PWR077
+L GND #PWR6021
 U 1 1 58A3787F
 P 4100 4700
-F 0 "#PWR077" H 4100 4450 50  0001 C CNN
+F 0 "#PWR6021" H 4100 4450 50  0001 C CNN
 F 1 "GND" H 4105 4527 50  0000 C CNN
 F 2 "" H 4100 4700 50  0000 C CNN
@@
 NoConn ~ 6350 4600
 $Comp
-L GND #PWR078
+L GND #PWR6020
 U 1 1 58A378BA
 P 6650 4000
-F 0 "#PWR078" H -400 1150 50  0001 C CNN
+F 0 "#PWR6020" H -400 1150 50  0001 C CNN
 F 1 "GND" V 6655 3872 50  0000 R CNN
 F 2 "" H -400 1400 50  0001 C CNN
@@
 $EndComp
 $Comp
-L GND #PWR079
+L GND #PWR6019
 U 1 1 58A39053
 P 5750 4000
-F 0 "#PWR079" H -1400 1650 50  0001 C CNN
+F 0 "#PWR6019" H -1400 1650 50  0001 C CNN
 F 1 "GND" V 5755 3872 50  0000 R CNN
 F 2 "" H -1400 1900 50  0001 C CNN
@@
 $EndComp
 $Comp
-L GND #PWR080
+L GND #PWR6006
 U 1 1 58A3B2B9
 P 3000 2350
-F 0 "#PWR080" H 50  -50 50  0001 C CNN
+F 0 "#PWR6006" H 50  -50 50  0001 C CNN
 F 1 "GND" V 3005 2222 50  0000 R CNN
 F 2 "" H 50  200 50  0001 C CNN
@@
 $EndComp
 $Comp
-L GND #PWR081
+L GND #PWR6016
 U 1 1 58A3B4D5
 P 3000 3800
-F 0 "#PWR081" H 50  1400 50  0001 C CNN
+F 0 "#PWR6016" H 50  1400 50  0001 C CNN
 F 1 "GND" V 3005 3672 50  0000 R CNN
 F 2 "" H 50  1650 50  0001 C CNN
@@
 $EndComp
 $Comp
-L VAA #PWR082
+L VAA #PWR6005
 U 1 1 58A8FF55
 P 6250 2250
-F 0 "#PWR082" H -2150 900 50  0001 C CNN
+F 0 "#PWR6005" H -2150 900 50  0001 C CNN
 F 1 "VAA" H 6267 2423 50  0000 C CNN
 F 2 "" H -2150 1050 50  0001 C CNN
@@
 $EndComp
 $Comp
-L VAA #PWR083
+L VAA #PWR6015
 U 1 1 58A9009E
 P 6250 3650
-F 0 "#PWR083" H -2150 2300 50  0001 C CNN
+F 0 "#PWR6015" H -2150 2300 50  0001 C CNN
 F 1 "VAA" H 6267 3823 50  0000 C CNN
 F 2 "" H -2150 2450 50  0001 C CNN
@@
 $EndComp
 $Comp
-L VAA #PWR084
+L VAA #PWR6001
 U 1 1 58A4CF7D
 P 5100 1800
-F 0 "#PWR084" H -3300 450 50  0001 C CNN
+F 0 "#PWR6001" H -3300 450 50  0001 C CNN
 F 1 "VAA" H 5117 1973 50  0000 C CNN
 F 2 "" H -3300 600 50  0001 C CNN
@@
 $EndComp
 $Comp
-L GND #PWR085
+L GND #PWR6002
 U 1 1 58A4D14E
 P 5100 2100
-F 0 "#PWR085" H 5100 1850 50  0001 C CNN
+F 0 "#PWR6002" H 5100 1850 50  0001 C CNN
 F 1 "GND" H 5105 1927 50  0000 C CNN
 F 2 "" H 5100 2100 50  0000 C CNN
@@
 $EndComp
 $Comp
-L GND #PWR086
+L GND #PWR6003
 U 1 1 58AB598A
 P 8700 2150
-F 0 "#PWR086" H 8750 2200 50  0001 C CNN
+F 0 "#PWR6003" H 8750 2200 50  0001 C CNN
 F 1 "GND" H 8705 1977 50  0000 C CNN
 F 2 "" H -1150 150 50  0001 C CNN
@@
 	8900 3700 10050 3700
 Wire Wire Line
-	4650 2900 5250 2900
+	5250 2900 4650 2900
 Connection ~ 4950 2900
 Wire Wire Line
 	4350 2900 4050 2900
 Wire Wire Line
-	5250 2900 5250 2800
+	5250 2750 5250 2900
 Wire Wire Line
 	5250 2800 6050 2800
@@
 	4100 4400 4100 4700
 Wire Wire Line
-	4650 4300 5250 4300
+	5250 4300 4650 4300
 Connection ~ 4950 4300
 Wire Wire Line
 	4350 4300 4050 4300
 Wire Wire Line
-	5250 4300 5250 4200
+	5250 4150 5250 4300
 Wire Wire Line
 	5250 4200 6050 4200
@@
 	8900 3700 8900 2150
 $Comp
-L GND #PWR087
+L GND #PWR6004
 U 1 1 58AB708B
 P 9100 2150
-F 0 "#PWR087" H 9150 2200 50  0001 C CNN
+F 0 "#PWR6004" H 9150 2200 50  0001 C CNN
 F 1 "GND" H 9105 1977 50  0000 C CNN
 F 2 "" H -750 150 50  0001 C CNN
@@
 	1    0    0    -1
 $EndComp
+$Comp
+L R R6001
+U 1 1 5910D830
+P 5250 2600
+F 0 "R6001" H 5320 2646 50  0000 L CNN
+F 1 "10k" H 5320 2555 50  0000 L CNN
+F 2 "Resistors_SMD:R_0805" V 5180 2600 50  0001 C CNN
+F 3 "" H 5250 2600 50  0001 C CNN
+	1    5250 2600
+	1    0    0    -1
+$EndComp
+$Comp
+L R R6002
+U 1 1 5910D890
+P 5250 4000
+F 0 "R6002" H 5320 4046 50  0000 L CNN
+F 1 "10k" H 5320 3955 50  0000 L CNN
+F 2 "Resistors_SMD:R_0805" V 5180 4000 50  0001 C CNN
+F 3 "" H 5250 4000 50  0001 C CNN
+	1    5250 4000
+	1    0    0    -1
+$EndComp
+$Comp
+L +3V3 #PWR6018
+U 1 1 5910D9E4
+P 5250 3850
+F 0 "#PWR6018" H 5250 3700 50  0001 C CNN
+F 1 "+3V3" H 5265 4023 50  0000 C CNN
+F 2 "" H 5250 3850 50  0001 C CNN
+F 3 "" H 5250 3850 50  0001 C CNN
+	1    5250 3850
+	1    0    0    -1
+$EndComp
+$Comp
+L +3V3 #PWR6008
+U 1 1 5910DA36
+P 5250 2450
+F 0 "#PWR6008" H 5250 2300 50  0001 C CNN
+F 1 "+3V3" H 5265 2623 50  0000 C CNN
+F 2 "" H 5250 2450 50  0001 C CNN
+F 3 "" H 5250 2450 50  0001 C CNN
+	1    5250 2450
+	1    0    0    -1
+$EndComp
+Connection ~ 5250 2800
+Connection ~ 5250 4200
 $EndSCHEMATC
