File: peripheral-board/audio.sch (KiCad schematic (older format))
At the start: 32 parts, among them J7001 FCR1295, J7002 53047-0310, U7001 LM386, U7002 LM386, U7003 MCP4011, U7004 MCP4011

Commit message: more audio circuit fixes
Parts:
- removed C7007, C7014: 1u, Capacitors_SMD:C_1206, symbol C
- R6001, R6002: value 10k -> 0; footprint Resistors_SMD:R_0805 -> Resistors_SMD:R_1206
Connections:
- net +3V3: no longer R6001.1, R6002.1
- net L: now also R6001.1
- net R: now also R6002.1
- net at U7003.3 (A): now also R6001.2
- net at U7004.3 (A): now also R6002.2
- net at C7009.1, R7003.1, R7004.1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: no longer R6001.2
- net at C7016.1, R7007.1, R7008.1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: no longer R6002.2
Changed lines of the file:
@@
 $EndComp
 $Comp
-L GND #PWR6014
+L GND #PWR068
 U 1 1 5823647F
 P 3300 3450
-F 0 "#PWR6014" H 3300 3200 50  0001 C CNN
+F 0 "#PWR068" H 3300 3200 50  0001 C CNN
 F 1 "GND" H 3305 3277 50  0000 C CNN
 F 2 "" H 3300 3450 50  0000 C CNN
@@
 $EndComp
 $Comp
-L GND #PWR6022
+L GND #PWR069
 U 1 1 582364AF
 P 3300 4850
-F 0 "#PWR6022" H 3300 4600 50  0001 C CNN
+F 0 "#PWR069" H 3300 4600 50  0001 C CNN
 F 1 "GND" H 3305 4677 50  0000 C CNN
 F 2 "" H 3300 4850 50  0000 C CNN
@@
 $EndComp
 $Comp
-L +3V3 #PWR6007
+L +3V3 #PWR070
 U 1 1 582364E9
 P 3300 2350
-F 0 "#PWR6007" H 3300 2200 50  0001 C CNN
+F 0 "#PWR070" H 3300 2200 50  0001 C CNN
 F 1 "+3V3" V 3315 2478 50  0000 L CNN
 F 2 "" H 3300 2350 50  0000 C CNN
@@
 $EndComp
 $Comp
-L +3V3 #PWR6017
+L +3V3 #PWR071
 U 1 1 58236543
 P 3350 3800
-F 0 "#PWR6017" H 3350 3650 50  0001 C CNN
+F 0 "#PWR071" H 3350 3650 50  0001 C CNN
 F 1 "+3V3" V 3365 3928 50  0000 L CNN
 F 2 "" H 3350 3800 50  0000 C CNN
@@
 DETECT
 $Comp
-L GND #PWR6012
+L GND #PWR072
 U 1 1 58240DA5
 P 4100 3300
-F 0 "#PWR6012" H 4100 3050 50  0001 C CNN
+F 0 "#PWR072" H 4100 3050 50  0001 C CNN
 F 1 "GND" H 4105 3127 50  0000 C CNN
 F 2 "" H 4100 3300 50  0000 C CNN
@@
 $EndComp
 $Comp
-L GND #PWR6013
+L GND #PWR073
 U 1 1 58A1A8BA
 P 10050 3400
-F 0 "#PWR6013" H 10100 3450 50  0001 C CNN
+F 0 "#PWR073" H 10100 3450 50  0001 C CNN
 F 1 "GND" V 10055 3272 50  0000 R CNN
 F 2 "" H 1200 200 50  0001 C CNN
@@
 $EndComp
 $Comp
-L +3V3 #PWR6011
+L +3V3 #PWR074
 U 1 1 58A1A914
 P 9950 3000
-F 0 "#PWR6011" H 10000 3050 50  0001 C CNN
+F 0 "#PWR074" H 10000 3050 50  0001 C CNN
 F 1 "+3V3" V 9965 3128 50  0000 L CNN
 F 2 "" H 1550 -100 50  0001 C CNN
@@
 $EndComp
 $Comp
-L C C7007
-U 1 1 58A34FD2
-P 4100 2650
-F 0 "C7007" H 3985 2604 50  0000 R CNN
-F 1 "1u" H 3985 2695 50  0000 R CNN
-F 2 "Capacitors_SMD:C_1206" H -912 -350 50  0001 C CNN
-F 3 "" H -950 -200 50  0001 C CNN
-	1    4100 2650
-	-1   0    0    1
-$EndComp
-$Comp
 L R R7003
 U 1 1 58A3508E
@@
 NoConn ~ 6350 3200
 $Comp
-L GND #PWR6010
+L GND #PWR075
 U 1 1 58A359F1
 P 6650 2600
-F 0 "#PWR6010" H -400 -250 50  0001 C CNN
+F 0 "#PWR075" H -400 -250 50  0001 C CNN
 F 1 "GND" V 6655 2472 50  0000 R CNN
 F 2 "" H -400 0   50  0001 C CNN
@@
 $EndComp
 $Comp
-L GND #PWR6009
+L GND #PWR076
 U 1 1 58A36C12
 P 5750 2600
-F 0 "#PWR6009" H -1400 250 50  0001 C CNN
+F 0 "#PWR076" H -1400 250 50  0001 C CNN
 F 1 "GND" V 5755 2472 50  0000 R CNN
 F 2 "" H -1400 500 50  0001 C CNN
@@
 $EndComp
 $Comp
-L GND #PWR6021
+L GND #PWR077
 U 1 1 58A3787F
 P 4100 4700
-F 0 "#PWR6021" H 4100 4450 50  0001 C CNN
+F 0 "#PWR077" H 4100 4450 50  0001 C CNN
 F 1 "GND" H 4105 4527 50  0000 C CNN
 F 2 "" H 4100 4700 50  0000 C CNN
@@
 $EndComp
 $Comp
-L C C7014
-U 1 1 58A3788B
-P 4100 4050
-F 0 "C7014" H 3985 4004 50  0000 R CNN
-F 1 "1u" H 3985 4095 50  0000 R CNN
-F 2 "Capacitors_SMD:C_1206" H -912 1050 50  0001 C CNN
-F 3 "" H -950 1200 50  0001 C CNN
-	1    4100 4050
-	-1   0    0    1
-$EndComp
-$Comp
 L R R7007
 U 1 1 58A37891
@@
 NoConn ~ 6350 4600
 $Comp
-L GND #PWR6020
+L GND #PWR078
 U 1 1 58A378BA
 P 6650 4000
-F 0 "#PWR6020" H -400 1150 50  0001 C CNN
+F 0 "#PWR078" H -400 1150 50  0001 C CNN
 F 1 "GND" V 6655 3872 50  0000 R CNN
 F 2 "" H -400 1400 50  0001 C CNN
@@
 $EndComp
 $Comp
-L GND #PWR6019
+L GND #PWR079
 U 1 1 58A39053
 P 5750 4000
-F 0 "#PWR6019" H -1400 1650 50  0001 C CNN
+F 0 "#PWR079" H -1400 1650 50  0001 C CNN
 F 1 "GND" V 5755 3872 50  0000 R CNN
 F 2 "" H -1400 1900 50  0001 C CNN
@@
 $EndComp
 $Comp
-L GND #PWR6006
+L GND #PWR080
 U 1 1 58A3B2B9
 P 3000 2350
-F 0 "#PWR6006" H 50  -50 50  0001 C CNN
+F 0 "#PWR080" H 50  -50 50  0001 C CNN
 F 1 "GND" V 3005 2222 50  0000 R CNN
 F 2 "" H 50  200 50  0001 C CNN
@@
 $EndComp
 $Comp
-L GND #PWR6016
+L GND #PWR081
 U 1 1 58A3B4D5
 P 3000 3800
-F 0 "#PWR6016" H 50  1400 50  0001 C CNN
+F 0 "#PWR081" H 50  1400 50  0001 C CNN
 F 1 "GND" V 3005 3672 50  0000 R CNN
 F 2 "" H 50  1650 50  0001 C CNN
@@
 $EndComp
 $Comp
-L VAA #PWR6005
+L VAA #PWR082
 U 1 1 58A8FF55
 P 6250 2250
-F 0 "#PWR6005" H -2150 900 50  0001 C CNN
+F 0 "#PWR082" H -2150 900 50  0001 C CNN
 F 1 "VAA" H 6267 2423 50  0000 C CNN
 F 2 "" H -2150 1050 50  0001 C CNN
@@
 $EndComp
 $Comp
-L VAA #PWR6015
+L VAA #PWR083
 U 1 1 58A9009E
 P 6250 3650
-F 0 "#PWR6015" H -2150 2300 50  0001 C CNN
+F 0 "#PWR083" H -2150 2300 50  0001 C CNN
 F 1 "VAA" H 6267 3823 50  0000 C CNN
 F 2 "" H -2150 2450 50  0001 C CNN
@@
 $EndComp
 $Comp
-L VAA #PWR6001
+L VAA #PWR084
 U 1 1 58A4CF7D
 P 5100 1800
-F 0 "#PWR6001" H -3300 450 50  0001 C CNN
+F 0 "#PWR084" H -3300 450 50  0001 C CNN
 F 1 "VAA" H 5117 1973 50  0000 C CNN
 F 2 "" H -3300 600 50  0001 C CNN
@@
 $EndComp
 $Comp
-L GND #PWR6002
+L GND #PWR085
 U 1 1 58A4D14E
 P 5100 2100
-F 0 "#PWR6002" H 5100 1850 50  0001 C CNN
+F 0 "#PWR085" H 5100 1850 50  0001 C CNN
 F 1 "GND" H 5105 1927 50  0000 C CNN
 F 2 "" H 5100 2100 50  0000 C CNN
@@
 $EndComp
 $Comp
-L GND #PWR6003
+L GND #PWR086
 U 1 1 58AB598A
 P 8700 2150
-F 0 "#PWR6003" H 8750 2200 50  0001 C CNN
+F 0 "#PWR086" H 8750 2200 50  0001 C CNN
 F 1 "GND" H 8705 1977 50  0000 C CNN
 F 2 "" H -1150 150 50  0001 C CNN
@@
 	4350 2900 4050 2900
 Wire Wire Line
-	5250 2750 5250 2900
-Wire Wire Line
 	5250 2800 6050 2800
 Connection ~ 5250 2900
@@
 	4350 4300 4050 4300
 Wire Wire Line
-	5250 4150 5250 4300
-Wire Wire Line
 	5250 4200 6050 4200
 Connection ~ 5250 4300
@@
 	8900 3700 8900 2150
 $Comp
-L GND #PWR6004
+L GND #PWR087
 U 1 1 58AB708B
 P 9100 2150
-F 0 "#PWR6004" H 9150 2200 50  0001 C CNN
+F 0 "#PWR087" H 9150 2200 50  0001 C CNN
 F 1 "GND" H 9105 1977 50  0000 C CNN
 F 2 "" H -750 150 50  0001 C CNN
@@
 	1    0    0    -1
 $EndComp
+Wire Wire Line
+	5250 2800 5250 2900
+Wire Wire Line
+	5250 4200 5250 4300
+$Comp
+L R R6002
+U 1 1 5910CA44
+P 4100 4050
+F 0 "R6002" H 4170 4096 50  0000 L CNN
+F 1 "0" H 4170 4005 50  0000 L CNN
+F 2 "Resistors_SMD:R_1206" V 4030 4050 50  0001 C CNN
+F 3 "" H 4100 4050 50  0001 C CNN
+	1    4100 4050
+	1    0    0    -1
+$EndComp
 $Comp
 L R R6001
-U 1 1 5910D830
-P 5250 2600
-F 0 "R6001" H 5320 2646 50  0000 L CNN
-F 1 "10k" H 5320 2555 50  0000 L CNN
-F 2 "Resistors_SMD:R_0805" V 5180 2600 50  0001 C CNN
-F 3 "" H 5250 2600 50  0001 C CNN
-	1    5250 2600
-	1    0    0    -1
-$EndComp
-$Comp
-L R R6002
-U 1 1 5910D890
-P 5250 4000
-F 0 "R6002" H 5320 4046 50  0000 L CNN
-F 1 "10k" H 5320 3955 50  0000 L CNN
-F 2 "Resistors_SMD:R_0805" V 5180 4000 50  0001 C CNN
-F 3 "" H 5250 4000 50  0001 C CNN
-	1    5250 4000
-	1    0    0    -1
-$EndComp
-$Comp
-L +3V3 #PWR6018
-U 1 1 5910D9E4
-P 5250 3850
-F 0 "#PWR6018" H 5250 3700 50  0001 C CNN
-F 1 "+3V3" H 5265 4023 50  0000 C CNN
-F 2 "" H 5250 3850 50  0001 C CNN
-F 3 "" H 5250 3850 50  0001 C CNN
-	1    5250 3850
-	1    0    0    -1
-$EndComp
-$Comp
-L +3V3 #PWR6008
-U 1 1 5910DA36
-P 5250 2450
-F 0 "#PWR6008" H 5250 2300 50  0001 C CNN
-F 1 "+3V3" H 5265 2623 50  0000 C CNN
-F 2 "" H 5250 2450 50  0001 C CNN
-F 3 "" H 5250 2450 50  0001 C CNN
-	1    5250 2450
-	1    0    0    -1
-$EndComp
-Connection ~ 5250 2800
-Connection ~ 5250 4200
+U 1 1 5910CC6F
+P 4100 2650
+F 0 "R6001" H 4170 2696 50  0000 L CNN
+F 1 "0" H 4170 2605 50  0000 L CNN
+F 2 "Resistors_SMD:R_1206" V 4030 2650 50  0001 C CNN
+F 3 "" H 4100 2650 50  0001 C CNN
+	1    4100 2650
+	1    0    0    -1
+$EndComp
 $EndSCHEMATC
