File: peripheral-board/keyboard.sch (KiCad schematic (older format))
At the start: 141 parts, among them SW2001 1, SW2002 2, SW2003 3, SW2004 4, SW2005 5, SW2006 6, SW2007 7, SW2008 8, SW2009 9, SW2010 0, SW2011 +, SW2012 ´, SW2013 BKSP, SW2014 TROLL, SW2015 §, SW2016 UP, SW2017 RMB, SW2018 Q, SW2019 W, SW2020 E, SW2021 R, SW2022 T, SW2023 Y, SW2024 U, SW2025 I, SW2026 O, SW2027 P, SW2028 Å, SW2029 ¨, SW2030 RETURN, SW2031 ALT_GR, SW2032 <, SW2033 LEFT, SW2034 MMB, SW2035 A, SW2036 S, SW2037 D, SW2038 F, SW2039 G, SW2040 H, SW2041 J, SW2042 K, SW2043 L, SW2044 Ö, SW2045 Ä, SW2046 ', SW2047 ESC, SW2048 TAB, SW2049 ALT, SW2050 DOWN, SW2051 LMB, SW2052 SHIFT_L, SW2053 Z, SW2054 X, SW2055 C, SW2056 V, SW2057 B, SW2058 N, SW2059 M, SW2060 ,, SW2061 ., SW2062 -, SW2063 SHIFT_R, SW2064 FN_R, SW2065 SPACE, SW2066 FN_L, SW2067 RIGHT, SW2068 CTRL, SW2069 SPACE, U2001 4017, U2002 4017, U2003 74HC00

Commit message: audio circuitry
Parts:
- RP2001: symbol R_PACK4 -> R_Pack04
- SW2001, SW2002, SW2003, SW2004, SW2005, SW2006, SW2007, SW2008, SW2009, SW2010, SW2011, SW2012, SW2013, SW2014, SW2015, SW2016, SW2017, SW2018, SW2019, SW2020, SW2021, SW2022, SW2023, SW2024, SW2025, SW2026, SW2027, SW2028, SW2029, SW2030, SW2031, SW2032, SW2033, SW2034, SW2035, SW2036, SW2037, SW2038, SW2039, SW2040, SW2041, SW2042, SW2043, SW2044, SW2045, SW2046, SW2047, SW2048, SW2049, SW2050, SW2051, SW2052, SW2053, SW2054, SW2055, SW2056, SW2057, SW2058, SW2059, SW2060, SW2061, SW2062, SW2063, SW2064, SW2065, SW2066, SW2067, SW2068, SW2069: symbol SW_PUSH_Small -> SW_Push_45deg

Commit message: routed traces.
Parts:
- D2001, D2002, D2003, D2004, D2005, D2006, D2007, D2008, D2009, D2010, D2011, D2012, D2013, D2014, D2015, D2016, D2017, D2018, D2019, D2020, D2021, D2022, D2023, D2024, D2025, D2026, D2027, D2028, D2029, D2030, D2031, D2032, D2033, D2034, D2035, D2036, D2037, D2038, D2039, D2040, D2041, D2042, D2043, D2044, D2045, D2046, D2047, D2048, D2049, D2050, D2051, D2052, D2053, D2054, D2055, D2056, D2057, D2058, D2059, D2060, D2061, D2062, D2063, D2064, D2065, D2066, D2067, D2068: footprint Diodes_SMD:MiniMELF_Standard -> Diodes_SMD:D_MiniMELF_Standard
